File: button.kicad_sch (KiCad schematic)
At the start: 4 parts, among them SW1 SW_Push

Commit message: working on the PCB
Parts:
- renumbered C10 to C14, R13 to R42, R14 to R43, SW1 to SW5
Changed lines of the file:
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@@
   (symbol (lib_id "power:GND") (at 108.585 89.535 0)
     (in_bom yes) (on_board yes) (fields_autoplaced)
-    (property "Reference" "#PWR031" (id 0) (at 108.585 95.885 0)
+    (property "Reference" "#PWR067" (id 0) (at 108.585 95.885 0)
       (effects (font (size 1.27 1.27)) hide)
     )
@@
   (symbol (lib_id "Switch:SW_Push") (at 108.585 82.55 270)
     (in_bom yes) (on_board yes) (fields_autoplaced)
-    (property "Reference" "SW1" (id 0) (at 113.03 81.2799 90)
+    (property "Reference" "SW5" (id 0) (at 113.03 81.2799 90)
       (effects (font (size 1.27 1.27)) (justify left))
     )
@@
   (symbol (lib_id "eurorack:R-10k-1206") (at 108.585 71.755 0)
     (in_bom yes) (on_board yes) (fields_autoplaced)
-    (property "Reference" "R14" (id 0) (at 110.49 70.4849 0)
+    (property "Reference" "R43" (id 0) (at 110.49 70.4849 0)
       (effects (font (size 1.27 1.27)) (justify left))
     )
@@
   (symbol (lib_id "eurorack:C-100nF-0805") (at 96.52 83.185 0)
     (in_bom yes) (on_board yes)
-    (property "Reference" "C10" (id 0) (at 97.79 85.725 0)
+    (property "Reference" "C14" (id 0) (at 97.79 85.725 0)
       (effects (font (size 1.27 1.27)) (justify left))
     )
@@
   (symbol (lib_id "power:+3V3") (at 108.585 66.04 0)
     (in_bom yes) (on_board yes) (fields_autoplaced)
-    (property "Reference" "#PWR030" (id 0) (at 108.585 69.85 0)
+    (property "Reference" "#PWR066" (id 0) (at 108.585 69.85 0)
       (effects (font (size 1.27 1.27)) hide)
     )
@@
   (symbol (lib_id "eurorack:R-100-1206") (at 102.87 77.47 270)
     (in_bom yes) (on_board yes)
-    (property "Reference" "R13" (id 0) (at 101.6 80.01 90))
+    (property "Reference" "R42" (id 0) (at 101.6 80.01 90))
     (property "Value" "R-100-1206" (id 1) (at 99.06 74.93 90))
     (property "Footprint" "Resistor_SMD:R_1206_3216Metric_Pad1.30x1.75mm_HandSolder" (id 2) (at 102.87 75.692 90)

Commit message: working on PCB, new iteratrion
Parts:
- renumbered C14 to C15, R42 to R44, R43 to R45, SW5 to SW6
Changed lines of the file:
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@@
   (symbol (lib_id "Switch:SW_Push") (at 108.585 82.55 270)
     (in_bom yes) (on_board yes) (fields_autoplaced)
-    (property "Reference" "SW5" (id 0) (at 113.03 81.2799 90)
+    (property "Reference" "SW6" (id 0) (at 113.03 81.2799 90)
       (effects (font (size 1.27 1.27)) (justify left))
     )
@@
   (symbol (lib_id "eurorack:R-10k-1206") (at 108.585 71.755 0)
     (in_bom yes) (on_board yes) (fields_autoplaced)
-    (property "Reference" "R43" (id 0) (at 110.49 70.4849 0)
+    (property "Reference" "R45" (id 0) (at 110.49 70.4849 0)
       (effects (font (size 1.27 1.27)) (justify left))
     )
@@
   (symbol (lib_id "eurorack:C-100nF-0805") (at 96.52 83.185 0)
     (in_bom yes) (on_board yes)
-    (property "Reference" "C14" (id 0) (at 97.79 85.725 0)
+    (property "Reference" "C15" (id 0) (at 97.79 85.725 0)
       (effects (font (size 1.27 1.27)) (justify left))
     )
@@
   (symbol (lib_id "eurorack:R-100-1206") (at 102.87 77.47 270)
     (in_bom yes) (on_board yes)
-    (property "Reference" "R42" (id 0) (at 101.6 80.01 90))
+    (property "Reference" "R44" (id 0) (at 101.6 80.01 90))
     (property "Value" "R-100-1206" (id 1) (at 99.06 74.93 90))
     (property "Footprint" "Resistor_SMD:R_1206_3216Metric_Pad1.30x1.75mm_HandSolder" (id 2) (at 102.87 75.692 90)

Commit message: working on the PCB
Parts:
- renumbered C15 to C11, R44 to R30, R45 to R31, SW6 to SW2
Changed lines of the file:
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@@
     (effects (font (size 1.27 1.27)) (justify right))
   )
-  (symbol (lib_id "power:GND") (at 108.585 89.535 0)
+  (symbol (lib_id "power:GND") (at 108.585 89.535 0) (unit 1)
     (in_bom yes) (on_board yes) (fields_autoplaced)
-    (property "Reference" "#PWR069" (id 0) (at 108.585 95.885 0)
+    (property "Reference" "#PWR053" (id 0) (at 108.585 95.885 0)
       (effects (font (size 1.27 1.27)) hide)
     )
@@
     (pin "1")
   )
-  (symbol (lib_id "Switch:SW_Push") (at 108.585 82.55 270)
+  (symbol (lib_id "Switch:SW_Push") (at 108.585 82.55 270) (unit 1)
     (in_bom yes) (on_board yes) (fields_autoplaced)
-    (property "Reference" "SW6" (id 0) (at 113.03 81.2799 90)
+    (property "Reference" "SW2" (id 0) (at 113.03 81.2799 90)
       (effects (font (size 1.27 1.27)) (justify left))
     )
@@
     (pin "2")
   )
-  (symbol (lib_id "eurorack:R-10k-1206") (at 108.585 71.755 0)
+  (symbol (lib_id "eurorack:R-10k-1206") (at 108.585 71.755 0) (unit 1)
     (in_bom yes) (on_board yes) (fields_autoplaced)
-    (property "Reference" "R45" (id 0) (at 110.49 70.4849 0)
+    (property "Reference" "R31" (id 0) (at 110.49 70.4849 0)
       (effects (font (size 1.27 1.27)) (justify left))
     )
@@
     (pin "2")
   )
-  (symbol (lib_id "eurorack:C-100nF-0805") (at 96.52 83.185 0)
+  (symbol (lib_id "eurorack:C-100nF-0805") (at 96.52 83.185 0) (unit 1)
     (in_bom yes) (on_board yes)
-    (property "Reference" "C15" (id 0) (at 97.79 85.725 0)
+    (property "Reference" "C11" (id 0) (at 97.79 85.725 0)
       (effects (font (size 1.27 1.27)) (justify left))
     )
@@
     (pin "2")
   )
-  (symbol (lib_id "power:+3V3") (at 108.585 66.04 0)
+  (symbol (lib_id "power:+3V3") (at 108.585 66.04 0) (unit 1)
     (in_bom yes) (on_board yes) (fields_autoplaced)
-    (property "Reference" "#PWR068" (id 0) (at 108.585 69.85 0)
+    (property "Reference" "#PWR052" (id 0) (at 108.585 69.85 0)
       (effects (font (size 1.27 1.27)) hide)
     )
@@
     (pin "1")
   )
-  (symbol (lib_id "eurorack:R-100-1206") (at 102.87 77.47 270)
+  (symbol (lib_id "eurorack:R-100-1206") (at 102.87 77.47 270) (unit 1)
     (in_bom yes) (on_board yes)
-    (property "Reference" "R44" (id 0) (at 101.6 80.01 90))
+    (property "Reference" "R30" (id 0) (at 101.6 80.01 90))
     (property "Value" "R-100-1206" (id 1) (at 99.06 74.93 90))
     (property "Footprint" "Resistor_SMD:R_1206_3216Metric_Pad1.30x1.75mm_HandSolder" (id 2) (at 102.87 75.692 90)

Commit message: yet an other new version with 3 boards
Connections:
- net GND renamed GND3
Changed lines of the file:
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@@
     (effects (font (size 1.27 1.27)) (justify right))
-  )
-  (symbol (lib_id "power:GND") (at 108.585 89.535 0) (unit 1)
-    (in_bom yes) (on_board yes) (fields_autoplaced)
-    (property "Reference" "#PWR053" (id 0) (at 108.585 95.885 0)
-      (effects (font (size 1.27 1.27)) hide)
-    )
-    (property "Value" "GND" (id 1) (at 108.585 93.98 0))
-    (property "Footprint" "" (id 2) (at 108.585 89.535 0)
-      (effects (font (size 1.27 1.27)) hide)
-    )
-    (property "Datasheet" "" (id 3) (at 108.585 89.535 0)
-      (effects (font (size 1.27 1.27)) hide)
-    )
-    (pin "1")
   )
   (symbol (lib_id "Switch:SW_Push") (at 108.585 82.55 270) (unit 1)
@@
     (pin "2")
   )
+  (symbol (lib_id "power:GND3") (at 108.585 89.535 0) (unit 1)
+    (in_bom yes) (on_board yes) (fields_autoplaced)
+    (property "Reference" "#PWR0137" (id 0) (at 108.585 95.885 0)
+      (effects (font (size 1.27 1.27)) hide)
+    )
+    (property "Value" "GND3" (id 1) (at 108.585 93.98 0))
+    (property "Footprint" "" (id 2) (at 108.585 89.535 0)
+      (effects (font (size 1.27 1.27)) hide)
+    )
+    (property "Datasheet" "" (id 3) (at 108.585 89.535 0)
+      (effects (font (size 1.27 1.27)) hide)
+    )
+    (pin "1")
+  )
   (symbol (lib_id "eurorack:R-10k-1206") (at 108.585 71.755 0) (unit 1)

Commit message: wip v3
Connections:
- net +3V3 renamed +3.3VA
Changed lines of the file:
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@@
     (pin "2")
+  )
+  (symbol (lib_id "power:+3.3VA") (at 108.585 66.04 0) (unit 1)
+    (in_bom yes) (on_board yes) (fields_autoplaced)
+    (property "Reference" "#PWR0172" (id 0) (at 108.585 69.85 0)
+      (effects (font (size 1.27 1.27)) hide)
+    )
+    (property "Value" "+3.3VA" (id 1) (at 108.585 60.96 0))
+    (property "Footprint" "" (id 2) (at 108.585 66.04 0)
+      (effects (font (size 1.27 1.27)) hide)
+    )
+    (property "Datasheet" "" (id 3) (at 108.585 66.04 0)
+      (effects (font (size 1.27 1.27)) hide)
+    )
+    (pin "1")
   )
   (symbol (lib_id "eurorack:C-100nF-0805") (at 96.52 83.185 0) (unit 1)
@@
     (pin "2")
   )
-  (symbol (lib_id "power:+3V3") (at 108.585 66.04 0) (unit 1)
-    (in_bom yes) (on_board yes) (fields_autoplaced)
-    (property "Reference" "#PWR052" (id 0) (at 108.585 69.85 0)
-      (effects (font (size 1.27 1.27)) hide)
-    )
-    (property "Value" "+3V3" (id 1) (at 108.585 60.96 0))
-    (property "Footprint" "" (id 2) (at 108.585 66.04 0)
-      (effects (font (size 1.27 1.27)) hide)
-    )
-    (property "Datasheet" "" (id 3) (at 108.585 66.04 0)
-      (effects (font (size 1.27 1.27)) hide)
-    )
-    (pin "1")
-  )
   (symbol (lib_id "eurorack:R-100-1206") (at 102.87 77.47 270) (unit 1)
