File: wt.kicad_pcb (KiCad board)
At the start: 4 copper layers, 91.3 x 100 mm, 182 parts, among them J1 USB_B, J2 Conn_ARM_JTAG_SWD_10, SW1 SW_Push, SW2 SW_Push, SW3 SW_Push, SW5 SW_Push, SW6 SW_Push, U1 LM324, U10 LUM-1502-03_3.5mm_mono_vertic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, U11 LUM-1502-03_3.5mm_mono_vertic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, U12 LUM-1502-03_3.5mm_mono_vertic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, U13 LUM-1502-03_3.5mm_mono_vertic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, U14 LUM-1502-03_3.5mm_mono_vertic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, U15 LUM-1502-03_3.5mm_mono_vertic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, U16 power_conn_10, U17 REF191, U18 L78L05ACU, U19 ZLDO1117G33TA, U2 LM324, U20 TL072, U21 LUM-1502-03_3.5mm_mono_vertic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, U22 LUM-1502-03_3.5mm_mono_vertic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, U23 LUM-1502-03_3.5mm_mono_vertic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, U24 LUM-1502-03_3.5mm_mono_vertic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, U3 LM324, U4 STM32F407VGTx, U5 TL074, U6 TL074, U7 TLC7528, U8 LUM-1502-03_3.5mm_mono_vertic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, U9 LUM-1502-03_3.5mm_mono_vertic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, Y1 Crystal_8Mhz

Commit message: working on the PCB
Parts:
- C1, C16, C17, C18, C19, C2, C20, C21, C22, C8, C9, D8, J2, JP1, JP2, R1, R10, R11, R12, R2, R4, R46, R47, R48, R5, R6, R7, R8, R9, RV9, U16, U17, U18, U19, U20, U3, U4, U5, U6, U7, Y1: moved to B.Cu
- moved Out_1 239.9 mm to (56.6, 94.0)
- moved Out_2 239.7 mm to (66.5, 94.0)
- moved R4 227.7 mm to (44.7, 48.5)
- moved R5 224.5 mm to (39.6, 37.4), turned to 90 degrees
- moved C9 224.3 mm to (24.9, 3.22)
- moved C3 223.2 mm to (79.2, 2.10)
- moved D28 223.2 mm to (118.4, 41.2)
- moved D7 223.2 mm to (118.4, 61.7)
- moved R78 223.2 mm to (109.5, 96.7)
- moved D29 223.2 mm to (146.2, 38.0)
- moved D3 223.2 mm to (146.2, 58.5)
- moved D30 223.2 mm to (99.7, 96.6)
- moved R18 223.2 mm to (81.7, 98.3)
- moved R19 223.2 mm to (86.1, 98.3)
- moved R21 223.2 mm to (156.0, 58.7)
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- renumbered SWe to SW4
Routing:
- net Net-(RV9-Pad2): track 0.00 -> 82.3 mm
- net AIN3: track 0.00 -> 72.2 mm, vias 0 -> 1
- net Net-(R6-Pad2): track 0.00 -> 57.9 mm, vias 0 -> 2
- net AIN2: track 0.00 -> 57.0 mm, vias 0 -> 1
- net AIN7: track 0.00 -> 54.8 mm
- net AIN10: track 0.00 -> 51.4 mm
- net AIN8: track 0.00 -> 50.8 mm, vias 0 -> 1
- net BTN4: track 0.00 -> 45.7 mm, vias 0 -> 1
- net AIN1: track 0.00 -> 40.9 mm, vias 0 -> 1
- net AIN6: track 0.00 -> 39.6 mm
- net AIN11: track 0.00 -> 38.0 mm, vias 0 -> 1
- net BTN3: track 0.00 -> 32.6 mm, vias 0 -> 1
- net /D0: track 0.00 -> 32.5 mm
- net AIN9: track 0.00 -> 32.4 mm
- net Net-(R5-Pad2): track 0.00 -> 31.4 mm
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- added copper zone on B.Cu, net GND
- added copper zone on F.Cu, net GND
- added copper zone on In1.Cu, net GND
- added copper zone on In2.Cu, net GND
Other:
- board size 91.3 x 100 mm -> 70.9 x 100 mm
- board text added: "HP16"

Commit message: working on PCB
Parts:
- D1, D2, D28, R15, R16, R17, R18, R19, R20, R72, R73, R74, U1: moved to B.Cu
- moved R15 120.3 mm to (56.4, 46.6), turned to 180 degrees
- moved D1 116.3 mm to (52.2, 42.4), turned to 180 degrees
- moved R17 106.5 mm to (49.8, 48.8), turned to -90 degrees
- moved R16 91.9 mm to (49.8, 45.4), turned to -90 degrees
- moved D2 79.5 mm to (52.3, 53.5), turned to 180 degrees
- moved R20 70.0 mm to (50.4, 59.9), turned to -90 degrees
- moved R73 58.9 mm to (74.2, 33.9), turned to 180 degrees
- moved R19 55.0 mm to (50.4, 56.4), turned to -90 degrees
- moved R72 50.2 mm to (78.6, 33.9), turned to 180 degrees
- moved R18 47.1 mm to (56.7, 58.3), turned to 180 degrees
- moved U1 46.3 mm to (11.4, 60.6), turned to 180 degrees
- moved R74 41.5 mm to (83.0, 33.9), turned to 180 degrees
- moved D28 30.9 mm to (88.4, 33.7), turned to 180 degrees
Routing:
- net Net-(RV13-Pad1): track 1.27 -> 77.6 mm
- net Net-(RV8-Pad1): track 1.27 -> 63.5 mm, vias 0 -> 1
- net Net-(R16-Pad2): track 0.00 -> 48.8 mm, vias 0 -> 2
- net Net-(RV4-Pad1): track 0.00 -> 42.5 mm, vias 0 -> 1
- net Net-(R19-Pad2): track 0.00 -> 40.5 mm, vias 0 -> 2
- net Net-(RV11-Pad1): track 1.27 -> 23.9 mm, vias 0 -> 1
- net Net-(RV3-Pad1): track 0.00 -> 20.3 mm
- net Net-(RV12-Pad1): track 1.27 -> 16.3 mm, vias 0 -> 1
- net Net-(RV2-Pad1): track 0.00 -> 9.23 mm, vias 0 -> 1
- net Net-(RV1-Pad1): track 0.00 -> 8.78 mm
- net AIN8: track 50.8 -> 56.9 mm
- net Net-(D1-Pad1): track 0.00 -> 4.12 mm
- net Net-(D2-Pad1): track 0.00 -> 3.64 mm
- net Net-(R18-Pad2): track 0.00 -> 3.26 mm
- net Net-(R15-Pad2): track 0.00 -> 2.73 mm
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
Commit message: PCV WIP
Parts:
- D27, D29, D30, D5, D6, R27, R28, R29, R32, R33, R34, R67, R68, R69, R75, R76, R77, R78, R79, R80, U2: moved to B.Cu
- moved R67 103.5 mm to (59.7, 58.3)
- moved R68 101.7 mm to (64.0, 53.3), turned to 90 degrees
- moved R76 101.0 mm to (61.5, 17.8), turned to -90 degrees
- moved R75 97.7 mm to (59.5, 22.8)
- moved R7 95.5 mm to (21.7, 12.7), turned to -90 degrees
- moved R69 94.8 mm to (61.9, 51.5), turned to 90 degrees
- moved R77 89.2 mm to (64.3, 19.7)
- moved D27 87.1 mm to (67.0, 56.3), turned to 180 degrees
- moved D29 86.2 mm to (63.2, 14.9), turned to 180 degrees
- moved R32 85.8 mm to (59.8, 71.3)
- moved R79 83.0 mm to (63.3, 31.0), turned to 90 degrees
- moved R33 82.3 mm to (64.1, 65.3), turned to 90 degrees
- moved R80 80.7 mm to (62.4, 28.2), turned to 180 degrees
- moved R78 79.6 mm to (59.6, 34.6)
- moved U2 78.6 mm to (28.8, 22.8), turned to 180 degrees
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Routing:
- net Net-(R33-Pad2): track 0.00 -> 82.1 mm, vias 0 -> 2
- net Net-(R68-Pad2): track 0.00 -> 55.8 mm, vias 0 -> 2
- net Net-(R28-Pad2): track 0.00 -> 43.4 mm, vias 0 -> 2
- net Net-(R79-Pad2): track 0.00 -> 41.6 mm, vias 0 -> 2
- net Net-(R76-Pad2): track 0.00 -> 34.5 mm, vias 0 -> 2
- net Net-(R73-Pad2): track 0.00 -> 29.7 mm, vias 0 -> 2
- net Net-(D28-Pad1): track 0.00 -> 6.02 mm
- net Net-(D29-Pad1): track 0.00 -> 4.80 mm
- net Net-(D6-Pad1): track 0.00 -> 3.97 mm
- net Net-(R5-Pad2): track 31.4 -> 35.3 mm
- net Net-(D27-Pad1): track 0.00 -> 3.73 mm
- net Net-(D30-Pad1): track 0.00 -> 3.71 mm
- net Net-(D5-Pad2): track 0.00 -> 3.67 mm
- net Net-(D6-Pad2): track 0.00 -> 3.43 mm
- net Net-(R67-Pad2): track 0.00 -> 3.16 mm
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
Commit message: fixed aligments - check again
Parts:
- D3, R21, R22, R23: moved to B.Cu
- moved R22 106.8 mm to (54.0, 66.9), turned to 90 degrees
- moved R21 100.6 mm to (56.2, 71.3), turned to 180 degrees
- moved R23 100.0 mm to (51.9, 67.0), turned to -90 degrees
- moved D3 89.0 mm to (57.7, 68.1), turned to 180 degrees
- moved D26 0.14 mm to (30.9, 51.9)
- moved SW1 0.14 mm to (27.6, 60.9)
- moved SW6 0.14 mm to (27.6, 85.9)
- moved R66 0.13 mm to (36.0, 51.9)
- moved RV10 0.13 mm to (47.1, 67.7)
- moved RV6 0.13 mm to (47.1, 82.0)
- moved RV7 0.13 mm to (47.1, 96.4)
- moved RV11 0.13 mm to (47.1, 33.5)
- moved RV12 0.13 mm to (47.1, 16.1)
- moved RV5 0.13 mm to (47.1, 53.3)
Routing:
- net Net-(R22-Pad2): track 0.00 -> 55.0 mm, vias 0 -> 4
- net Net-(D3-Pad1): track 0.00 -> 3.81 mm
- net Net-(R21-Pad2): track 0.00 -> 2.37 mm
- net Net-(D3-Pad2): track 0.00 -> 2.11 mm

Commit message: working on PCB, new iteratrion
Parts:
- D4, D7, R24, R25, R26, R35, R36, R37, R70, R71: moved to B.Cu
- JP1, JP2: footprint Connector_PinSocket_2.54mm:PinSocket_1x03_P2.54mm_Vertical -> Jumper:SolderJumper-3_P1.3mm_Open_RoundedPad1.0x1.5mm
- moved R71 74.3 mm to (47.1, 8.51), turned to 45 degrees
- moved R35 71.7 mm to (59.6, 82.9)
- moved R36 71.1 mm to (63.6, 78.8), turned to 90 degrees
- moved R70 68.9 mm to (48.7, 10.2), turned to 45 degrees
- moved R37 64.5 mm to (61.5, 78.8), turned to -90 degrees
- moved C8 59.1 mm to (-37.8, 34.3)
- moved C9 59.1 mm to (-25.3, 34.4)
- moved R11 59.1 mm to (-20.3, 34.4)
- moved R12 59.1 mm to (-32.6, 34.4)
- moved R48 59.1 mm to (-8.81, 40.0)
- moved R7 59.1 mm to (-28.5, 43.8)
- moved R8 59.1 mm to (-40.8, 42.7)
- moved R10 59.1 mm to (-42.8, 34.3)
- moved R9 59.1 mm to (-16.6, 35.7)
- moved C3 58.7 mm to (21.3, 12.0), turned to 180 degrees
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Connections:
- net Net-(J1-Pad2) renamed D-
- net Net-(J1-Pad3) renamed D+
- net PA11 renamed USB_D-
- net PA12 renamed USB_D+
Routing:
- net LED14: track 0.00 -> 90.5 mm, vias 0 -> 1
- net Net-(RV9-Pad2): track 82.3 -> 0.00 mm
- net Net-(RV13-Pad1): track 77.6 -> 8.46 mm
- net Net-(R6-Pad2): track 57.9 -> 0.00 mm, vias 2 -> 0
- net LED13: track 0.00 -> 56.5 mm, vias 0 -> 1
- net Net-(R22-Pad2): track 55.0 -> 0.00 mm, vias 4 -> 0
- net AIN7: track 54.8 -> 108.3 mm, vias 0 -> 1
- net AIN5: track 24.7 -> 75.5 mm, vias 0 -> 1
- net AIN6: track 39.6 -> 89.9 mm, vias 0 -> 1
- net AIN4: track 11.6 -> 61.5 mm, vias 0 -> 1
- net Net-(R16-Pad2): track 48.8 -> 0.00 mm, vias 2 -> 0
- net Net-(RV7-Pad1): track 1.27 -> 48.1 mm, vias 0 -> 1
- net Net-(R36-Pad2): track 0.00 -> 46.3 mm
- net BTN4: track 45.7 -> 0.00 mm, vias 1 -> 0
- net Net-(RV8-Pad1): track 63.5 -> 20.9 mm, vias 1 -> 0
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
Commit message: working on the PCB
Parts:
- C17: moved to F.Cu
- C4, C5: footprint Capacitor_SMD:C_1812_4532Metric_Pad1.57x3.40mm_HandSolder -> Capacitor_SMD:C_0603_1608Metric; moved to B.Cu
- C6: moved to B.Cu
- moved R10 78.2 mm to (34.8, 43.8), turned to -90 degrees
- moved C5 75.9 mm to (42.1, 18.4)
- moved RV9 70.2 mm to (35.5, 76.4)
- moved R12 65.7 mm to (32.4, 43.8), turned to 90 degrees
- moved R8 63.1 mm to (21.4, 53.3), turned to 0 degrees
- moved C8 62.3 mm to (24.2, 40.0)
- moved C4 61.0 mm to (38.2, 4.52), turned to -45 degrees
- moved C17 52.1 mm to (-9.98, 42.2), turned to 0 degrees
- moved C6 51.2 mm to (20.8, 8.76), turned to -90 degrees
- moved R11 38.3 mm to (17.8, 38.6)
- moved R7 37.8 mm to (9.02, 48.1)
- moved C9 34.9 mm to (8.97, 41.1), turned to -90 degrees
- moved R9 29.5 mm to (12.8, 38.6), turned to 0 degrees
- moved C7 29.4 mm to (16.4, 10.4), turned to 90 degrees
- moved R48 18.7 mm to (6.76, 29.7), turned to -90 degrees
Routing:
- net /DCA/OutA: track 0.00 -> 105.4 mm, vias 0 -> 1
- net /DCA/OutB: track 0.00 -> 81.5 mm, vias 0 -> 1
- net BTN1: track 0.00 -> 80.3 mm, vias 0 -> 5
- net BTN0: track 0.00 -> 79.1 mm, vias 0 -> 5
- net BTN2: track 0.00 -> 78.1 mm, vias 0 -> 1
- net LED7: track 0.00 -> 75.3 mm, vias 0 -> 1
- net LED15: track 0.00 -> 56.3 mm, vias 0 -> 3
- net Net-(R25-Pad2): track 0.00 -> 56.1 mm, vias 0 -> 2
- net LED6: track 0.00 -> 48.3 mm, vias 0 -> 3
- net Net-(RV9-Pad2): track 0.00 -> 47.8 mm
- net Net-(C8-Pad2): track 0.00 -> 23.9 mm
- net Net-(C9-Pad1): track 0.00 -> 20.9 mm
- net Net-(R42-Pad1): track 0.00 -> 17.5 mm
- net Net-(C8-Pad1): track 0.00 -> 15.6 mm
- net +3V3: track 26.7 -> 38.8 mm, vias 0 -> 1
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
Commit message: working on the PCB
Parts:
- removed C17: C-Pol-10uF-FK-V, Capacitor_SMD:CP_Elec_8x6.2
- moved R6 30.2 mm to (16.3, 53.3), turned to 0 degrees
- moved R5 28.5 mm to (11.2, 36.2), turned to 0 degrees
- moved C4 1.87 mm to (39.6, 5.82)
Routing:
- net +3V3: track 38.8 -> 385.0 mm, vias 1 -> 24
- net +12V: track 32.8 -> 265.8 mm, vias 1 -> 9
- net JTDI: track 0.00 -> 92.9 mm, vias 0 -> 2
- net -12V: track 13.7 -> 104.2 mm, vias 0 -> 2
- net /DCA/InB: track 0.00 -> 81.1 mm, vias 0 -> 2
- net BTN3: track 2.22 -> 64.1 mm, vias 0 -> 3
- net /DCA/InA: track 0.00 -> 54.3 mm, vias 0 -> 2
- net Net-(R5-Pad2): track 3.38 -> 17.6 mm
- net LED7: track 75.3 -> 66.8 mm
- net SWDCLK: track 0.00 -> 4.70 mm
- net LED14: track 95.4 -> 90.8 mm
- net LED15: track 56.3 -> 53.4 mm
- net BTN1: track 80.3 -> 82.3 mm
- net Net-(R6-Pad2): track 6.13 -> 8.14 mm
- net Net-(C9-Pad1): track 20.9 -> 22.8 mm
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
Commit message: Working on the PCB / JTAG
Parts:
- moved JP1 2.37 mm to (21.6, 23.8), turned to -135 degrees
Routing:
- net TRACESWO: track 0.00 -> 108.0 mm, vias 0 -> 4
- net SWDCLK: track 4.70 -> 96.7 mm, vias 0 -> 2
- net GND: track 55.8 -> 72.2 mm, vias 1 -> 3
- net Net-(JP1-Pad2): track 3.63 -> 6.73 mm
- net AIN11: track 49.8 -> 51.5 mm
- net /DCA/OutA: track 105.4 -> 104.0 mm
- net Net-(U5-Pad13): track 0.00 -> 1.27 mm
- net Net-(D5-Pad1): track 2.91 -> 1.86 mm
- net Net-(R27-Pad2): track 2.46 -> 1.49 mm
- net AIN10: track 32.8 -> 31.9 mm
- net Net-(R72-Pad2): track 2.48 -> 1.64 mm
- net Net-(R13-Pad1): track 7.93 -> 7.11 mm
- net BTN0: track 78.6 -> 77.8 mm
- net Net-(R24-Pad2): track 2.46 -> 1.69 mm
- net Net-(R40-Pad1): track 7.55 -> 6.83 mm
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