File: wt.kicad_pcb (KiCad board)
At the start: 4 copper layers, 125 x 100 mm, 213 parts, among them J1 USB_B, J2 Conn_ARM_JTAG_SWD_10, SW1 SW_Push, SW2 SW_Push, SW3 SW_Push, SW4 SW_Push, SW5 SW_Push, SW6 SW_Push, U1 LM324, U10 LUM-1502-03_3.5mm_mono_vertic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, U11 LUM-1502-03_3.5mm_mono_vertic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, U12 LUM-1502-03_3.5mm_mono_vertic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, U13 LUM-1502-03_3.5mm_mono_vertic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, U14 LUM-1502-03_3.5mm_mono_vertic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, U15 LUM-1502-03_3.5mm_mono_vertic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, U16 power_conn_16, U17 REF191, U18 LM7805_TO220, U19 ZLDO1117G33TA, U2 LM324, U21 LUM-1502-03_3.5mm_mono_vertic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, U22 LUM-1502-03_3.5mm_mono_vertic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, U23 LUM-1502-03_3.5mm_mono_vertic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, U24 LUM-1502-03_3.5mm_mono_vertic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, U3 LM324, U4 STM32F407VGTx, U5 TL074, U6 TL074, U7 TLC7528, U8 LUM-1502-03_3.5mm_mono_vertic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, U9 LUM-1502-03_3.5mm_mono_vertic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, Y1 Crystal_8Mhz

Commit message: wip led panel
Parts:
- removed REF** (x12): mount_Potentiometer_Piher_PT-10-V10_Vertical, eurorack:mount_Potentiometer_Piher_PT-10-V10_Vertical
- removed REF** (x6): mount_SW_PUSH_6mm_H9.5mm, eurorack:mount_SW_PUSH_6mm_H9.5mm
- removed REF** (x14): mount_LUM_1502-03, eurorack:mount_LUM_1502-03
- removed REF**: mount_USB-BG, eurorack:mount_USB-BG
- added C26: C-100nF-0805, Capacitor_SMD:C_0805_2012Metric_Pad1.18x1.45mm_HandSolder, F.Cu at (5.44, -18.1)
- added C27: C-100nF-0805, Capacitor_SMD:C_0805_2012Metric_Pad1.18x1.45mm_HandSolder, F.Cu at (0.63, -18.1)
- added C28: C-100nF-0805, Capacitor_SMD:C_0805_2012Metric_Pad1.18x1.45mm_HandSolder, F.Cu at (63.4, -46.3)
- added C29: C-100nF-0805, Capacitor_SMD:C_0805_2012Metric_Pad1.18x1.45mm_HandSolder, F.Cu at (53.8, -43.3)
- added C30: C-100nF-0805, Capacitor_SMD:C_0805_2012Metric_Pad1.18x1.45mm_HandSolder, F.Cu at (63.4, -49.3)
- added C31: C-100nF-0805, Capacitor_SMD:C_0805_2012Metric_Pad1.18x1.45mm_HandSolder, F.Cu at (53.8, -46.3)
- added C32: C-100nF-0805, Capacitor_SMD:C_0805_2012Metric_Pad1.18x1.45mm_HandSolder, F.Cu at (58.6, -46.3)
- added C33: C-100nF-0805, Capacitor_SMD:C_0805_2012Metric_Pad1.18x1.45mm_HandSolder, F.Cu at (53.8, -40.2)
- added C34: C-100nF-0805, Capacitor_SMD:C_0805_2012Metric_Pad1.18x1.45mm_HandSolder, F.Cu at (58.6, -43.3)
- added C35: C-100nF-0805, Capacitor_SMD:C_0805_2012Metric_Pad1.18x1.45mm_HandSolder, F.Cu at (58.6, -49.3)
- added C36: C-100nF-0805, Capacitor_SMD:C_0805_2012Metric_Pad1.18x1.45mm_HandSolder, F.Cu at (53.8, -49.3)
- added C37: C-100nF-0805, Capacitor_SMD:C_0805_2012Metric_Pad1.18x1.45mm_HandSolder, F.Cu at (58.6, -32.5)
- added C38: C-100nF-0805, Capacitor_SMD:C_0805_2012Metric_Pad1.18x1.45mm_HandSolder, F.Cu at (53.8, -32.5)
- added C39: C-100nF-0805, Capacitor_SMD:C_0805_2012Metric_Pad1.18x1.45mm_HandSolder, F.Cu at (53.8, -29.5)
- added J3: Conn_01x10_Female, Connector_PinHeader_2.54mm:PinHeader_1x10_P2.54mm_Vertical, F.Cu at (91.2, 16.6)
- added J4: Conn_01x10_Male, Connector_PinHeader_2.54mm:PinHeader_2x05_P2.54mm_Vertical, F.Cu at (86.2, 47.4)
- added J5: Conn_01x10_Male, Connector_PinSocket_2.54mm:PinSocket_1x10_P2.54mm_Vertical, B.Cu at (118.2, 29.9)
- added J6: Conn_01x10_Female, Connector_PinSocket_2.54mm:PinSocket_2x05_P2.54mm_Vertical, B.Cu at (113.2, 44.9)
- moved C1 52.0 mm to (-39.6, 20.4)
- moved C17 52.0 mm to (-18.2, 41.2)
- moved C4 52.0 mm to (-11.5, 5.96)
- moved C5 52.0 mm to (-11.3, 20.4)
- moved C6 52.0 mm to (-31.7, 9.57)
- moved C8 52.0 mm to (-27.8, 41.2)
- moved C9 52.0 mm to (-43.0, 42.3)
- moved R10 52.0 mm to (-17.2, 44.9)
- moved R11 52.0 mm to (-34.2, 39.8)
- moved R12 52.0 mm to (-19.6, 44.9)
- moved R2 52.0 mm to (-39.8, 10.7)
- moved R4 52.0 mm to (-18.3, 2.81)
- moved R48 52.0 mm to (-45.3, 28.6)
- moved U1 52.0 mm to (-40.5, 62.1)
- moved U2 52.0 mm to (-14.8, 57.3)
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Connections:
- D10 pad 1: GND -> GND2
- D11 pad 1: GND -> GND2
- D12 pad 1: GND -> GND2
- D13 pad 1: GND -> GND2
- D14 pad 1: GND -> GND2
- D15 pad 1: GND -> GND2
- D16 pad 1: GND -> GND2
- D17 pad 1: GND -> GND2
- D18 pad 1: GND -> GND2
- D19 pad 1: GND -> GND2
- D20 pad 1: GND -> GND2
- D21 pad 1: GND -> GND2
- D22 pad 1: GND -> GND2
- D23 pad 1: GND -> GND2
- D24 pad 1: GND -> GND2
- D25 pad 1: GND -> GND2
- D26 pad 1: GND -> GND2
- D9 pad 1: GND -> GND2
- R49 pad 2: LED0 -> Net-(R49-Pad2)
- R50 pad 2: LED1 -> Net-(R50-Pad2)
- R51 pad 2: LED2 -> Net-(R51-Pad2)
- R52 pad 2: LED3 -> Net-(R52-Pad2)
- R53 pad 2: LED4 -> Net-(R53-Pad2)
- R54 pad 2: LED5 -> Net-(R54-Pad2)
- R55 pad 2: LED6 -> Net-(R55-Pad2)
- R56 pad 2: LED7 -> Net-(R56-Pad2)
- R57 pad 2: LED8 -> Net-(R57-Pad2)
- R58 pad 2: LED9 -> Net-(R58-Pad2)
- R59 pad 2: LED10 -> Net-(R59-Pad2)
- R60 pad 2: LED11 -> Net-(R60-Pad2)
- R61 pad 2: LED12 -> Net-(J6-Pad4)
- R62 pad 2: LED13 -> Net-(R62-Pad2)
- R63 pad 2: LED14 -> Net-(R63-Pad2)
- R64 pad 2: LED15 -> Net-(R64-Pad2)
- R65 pad 2: LED17 -> Net-(R65-Pad2)
- R66 pad 2: LED16 -> Net-(R66-Pad2)
Other:
- board size 125 x 100 mm -> 120 x 100.1 mm
- board text added: "WT-V003"
- board text removed: "WT-V002"

Commit message: working on v3 - todo go on with power lines
Parts:
- added G***: LOGO, eurorack:logo_small, B.Cu at (106.4, 9.30)
- added RV1: Pot_500, eurorack:Potentiometer_Piher_PT-10-V10_Vertical, F.Cu at (8.54, 53.3)
- added RV6: Pot_500, eurorack:Potentiometer_Piher_PT-10-V10_Vertical, F.Cu at (47.1, 82.0)
- C17, C23, C6, C8, C9, R10, R11, R12, R9, U3, U5, U6, U7: moved to F.Cu
- C3, R3: moved to B.Cu
- moved R48 98.6 mm to (52.7, 17.8), turned to 0 degrees
- moved U3 73.7 mm to (29.7, 5.92)
- moved R2 64.4 mm to (24.2, 3.23), turned to 180 degrees
- moved Y1 61.2 mm to (25.0, 6.93), turned to 180 degrees
- moved C2 59.8 mm to (18.7, 3.38), turned to 180 degrees
- moved C6 59.5 mm to (27.7, 11.7)
- moved U1 58.6 mm to (13.7, 39.8)
- moved C23 58.5 mm to (14.6, 35.1)
- moved C9 57.8 mm to (14.0, 32.8), turned to 0 degrees
- moved U6 57.6 mm to (27.8, 26.2)
- moved R9 57.5 mm to (17.9, 34.1), turned to -90 degrees
- moved U5 57.4 mm to (16.8, 26.2)
- moved J3 57.4 mm to (35.4, 30.0)
- moved C1 56.8 mm to (14.5, 3.39), turned to 180 degrees
- moved J4 55.8 mm to (30.4, 45.0), turned to -90 degrees
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Routing:
- net +3V3: track 0.00 -> 284.9 mm, vias 0 -> 16
- net +12V: track 0.00 -> 174.3 mm, vias 0 -> 1
- net +5V: track 0.00 -> 160.3 mm, vias 0 -> 2
- net /DCA/OutA: track 0.00 -> 102.7 mm
- net /DCA/OutB: track 0.00 -> 98.2 mm
- net AIN3: track 0.00 -> 93.9 mm, vias 0 -> 2
- net LED0: track 0.00 -> 87.3 mm, vias 0 -> 1
- net AIN7: track 0.00 -> 84.8 mm
- net AIN2: track 0.00 -> 78.4 mm, vias 0 -> 2
- net LED1: track 0.00 -> 76.3 mm, vias 0 -> 1
- net Net-(R22-Pad2): track 0.00 -> 76.0 mm, vias 0 -> 2
- net Net-(R25-Pad2): track 0.00 -> 75.3 mm, vias 0 -> 2
- net Net-(RV7-Pad1): track 0.00 -> 70.9 mm
- net PA9: track 0.00 -> 69.2 mm, vias 0 -> 2
- net Net-(RV13-Pad1): track 0.00 -> 68.4 mm
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Other:
- board size 120 x 100.1 mm -> 120 x 100 mm
- board text added: "5V Int"
- board text added: "LP-001"

Commit message: wip - go btn
Parts:
- moved R3 2.19 mm to (31.6, 10.1), turned to 90 degrees
- moved C3 0.82 mm to (29.9, 10.3), turned to -90 degrees
Routing:
- net -12V: track 6.81 -> 182.2 mm, vias 0 -> 2
- net 1V25: track 5.75 -> 119.3 mm, vias 0 -> 2
- net +12V: track 174.3 -> 259.3 mm, vias 1 -> 8
- net BTN4: track 5.70 -> 74.1 mm, vias 0 -> 4
- net BTN5: track 2.25 -> 69.3 mm, vias 0 -> 4
- net BTN0: track 2.34 -> 40.5 mm, vias 0 -> 2
- net BTN1: track 2.22 -> 39.2 mm, vias 0 -> 2
- net +3V3: track 284.9 -> 314.3 mm, vias 16 -> 15
- net AIN11-LED: track 4.72 -> 25.9 mm, vias 0 -> 2
- net LED4: track 27.8 -> 38.2 mm
- net RST: track 56.6 -> 47.2 mm
- net SWDCLK: track 26.0 -> 28.7 mm
- net LED1: track 76.3 -> 74.4 mm
- net LED0: track 87.3 -> 85.6 mm
- net SWDIO: track 14.4 -> 16.0 mm
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
Commit message: working on the v3 leds
Parts:
- moved R4 0.06 mm to (32.1, 24.7)
- moved R3 0.06 mm to (31.7, 10.1)
Routing:
- net AIN6-LED: track 4.72 -> 124.7 mm, vias 0 -> 6
- net AIN5-LED: track 4.72 -> 111.6 mm, vias 0 -> 4
- net AIN3-LED: track 4.72 -> 88.8 mm, vias 0 -> 1
- net AIN4-LED: track 4.72 -> 81.4 mm, vias 0 -> 2
- net AIN2-LED: track 4.72 -> 72.6 mm, vias 0 -> 1
- net BTN3: track 0.00 -> 55.9 mm, vias 0 -> 5
- net BTN2: track 5.12 -> 51.2 mm, vias 0 -> 3
- net Net-(R1-Pad2): track 0.00 -> 45.6 mm, vias 0 -> 3
- net RST: track 47.2 -> 71.2 mm
- net +3V3: track 314.3 -> 336.1 mm, vias 15 -> 17
- net 1V25: track 119.3 -> 131.6 mm
- net Net-(JP1-Pad2): track 0.00 -> 6.07 mm
- net LED0: track 85.6 -> 81.7 mm
- net AIN4: track 34.8 -> 36.6 mm
- net GND: track 14.1 -> 15.9 mm, vias 0 -> 1
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
Commit message: woking on the LEDs
Parts:
- R4: moved to F.Cu
- moved R4 6.98 mm to (29.1, 18.4), turned to 0 degrees
- moved C4 3.09 mm to (29.2, 30.6)
Routing:
- net AIN0-LED: track 6.46 -> 91.2 mm, vias 1 -> 2
- net AIN7-LED: track 4.72 -> 88.0 mm, vias 0 -> 3
- net AIN1-LED: track 4.72 -> 81.4 mm, vias 0 -> 5
- net -12V: track 182.8 -> 111.8 mm, vias 2 -> 3
- net LED17: track 0.00 -> 48.7 mm, vias 0 -> 1
- net TRACESWO: track 0.00 -> 44.7 mm
- net LED16: track 0.00 -> 42.7 mm, vias 0 -> 1
- net AIN9-LED: track 4.72 -> 42.9 mm, vias 0 -> 1
- net AIN10-LED: track 4.72 -> 38.4 mm, vias 0 -> 3
- net AIN8-LED: track 4.72 -> 36.1 mm, vias 0 -> 2
- net LED15: track 0.00 -> 11.1 mm, vias 0 -> 1
- net 1V25: track 131.6 -> 138.8 mm
- net +3V3: track 336.1 -> 341.4 mm, vias 17 -> 18
- net Net-(C17-Pad1): track 49.9 -> 44.7 mm
- net +12V: track 259.3 -> 255.4 mm, vias 8 -> 10
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
Commit message: yet an other new version with 3 boards
Parts:
- removed the RV1 at (8.54, 53.3)
- removed the RV6 at (47.1, 82.0)
- added BackBoard_1: Conn_01x28_Female, Connector_PinSocket_2.54mm:PinSocket_2x14_P2.54mm_Vertical, F.Cu at (31.8, -100.4)
- added BackBoard_2: Conn_01x14_Male, Connector_PinHeader_2.54mm:PinHeader_1x14_P2.54mm_Vertical, F.Cu at (13.2, -41.0)
- added BackBoard_3: Conn_01x14_Male, Connector_PinHeader_2.54mm:PinHeader_1x14_P2.54mm_Vertical, F.Cu at (37.2, -41.0)
- added FrontBoard_1: Conn_01x28_Male, Connector_PinHeader_2.54mm:PinHeader_2x14_P2.54mm_Vertical, B.Cu at (31.8, 4.60)
- added FrontBoard_2: Conn_01x14_Female, Connector_PinSocket_2.54mm:PinSocket_1x14_P2.54mm_Vertical, B.Cu at (13.2, 64.0)
- added FrontBoard_3: Conn_01x14_Female, Connector_PinSocket_2.54mm:PinSocket_1x14_P2.54mm_Vertical, B.Cu at (37.2, 64.0)
- C1, C2, C3, C5, R2, R3, Y1: moved to F.Cu
- U3: moved to B.Cu
- moved C4 212.1 mm to (207.9, -83.5), turned to 45 degrees
- moved U16 208.1 mm to (156.2, -69.8)
- moved C16 207.3 mm to (149.4, -97.3)
- moved C18 207.3 mm to (141.0, -93.0)
- moved C21 207.3 mm to (122.1, -85.0)
- moved C22 207.3 mm to (157.9, -83.0)
- moved C24 207.3 mm to (130.9, -86.6)
- moved C25 207.3 mm to (141.8, -86.8)
- moved JP2 207.3 mm to (121.1, -88.9)
- moved U17 207.3 mm to (146.0, -93.4)
- moved C19 207.3 mm to (138.9, -93.4)
- moved U19 207.3 mm to (150.4, -86.1)
- moved C5 182.5 mm to (182.4, -40.0), turned to 0 degrees
- moved J2 181.9 mm to (178.7, -50.7)
- moved U18 166.8 mm to (116.2, -60.9)
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Connections:
- C10 pad 2: GND -> GND3
- C11 pad 2: GND -> GND3
- C12 pad 2: GND -> GND3
- C13 pad 2: GND -> GND3
- C14 pad 2: GND -> GND3
- C15 pad 2: GND -> GND3
- C37 pad 2: GND -> GND3
- C38 pad 2: GND -> GND3
- C39 pad 2: GND -> GND3
- J3 pad 10: GND -> GND3
- J4 pad 10: GND -> GND3
- R17 pad 2: GND -> GND3
- R20 pad 2: GND -> GND3
- R23 pad 2: GND -> GND3
- R26 pad 2: GND -> GND3
- R29 pad 2: GND -> GND3
- R34 pad 2: GND -> GND3
- R37 pad 2: GND -> GND3
- R48 pad 2: GND -> GND3
- R69 pad 2: GND -> GND3
- R74 pad 2: GND -> GND3
- R77 pad 2: GND -> GND3
- R80 pad 2: GND -> GND3
- RV1 pad 11: GND -> GND3
- RV1 pad 3: GND -> GND3
- RV1 pad 7: GND -> GND3
- RV10 pad 11: GND -> GND3
- RV10 pad 3: GND -> GND3
- RV10 pad 7: GND -> GND3
- RV11 pad 11: GND -> GND3
- RV11 pad 3: GND -> GND3
- RV11 pad 7: GND -> GND3
- RV12 pad 11: GND -> GND3
- RV12 pad 3: GND -> GND3
- RV12 pad 7: GND -> GND3
- RV13 pad 11: GND -> GND3
- RV13 pad 3: GND -> GND3
- RV13 pad 7: GND -> GND3
- RV2 pad 11: GND -> GND3
- RV2 pad 3: GND -> GND3
- RV2 pad 7: GND -> GND3
- RV3 pad 11: GND -> GND3
- RV3 pad 3: GND -> GND3
- RV3 pad 7: GND -> GND3
- RV4 pad 11: GND -> GND3
- RV4 pad 3: GND -> GND3
- RV4 pad 7: GND -> GND3
- RV5 pad 11: GND -> GND3
- RV5 pad 3: GND -> GND3
- RV5 pad 7: GND -> GND3
- RV6 pad 11: GND -> GND3
- RV6 pad 3: GND -> GND3
- RV6 pad 7: GND -> GND3
- RV7 pad 11: GND -> GND3
- RV7 pad 3: GND -> GND3
- RV7 pad 7: GND -> GND3
- RV8 pad 11: GND -> GND3
- RV8 pad 3: GND -> GND3
- RV8 pad 7: GND -> GND3
- SW1 pad 2: GND -> GND3
- SW2 pad 2: GND -> GND3
- SW3 pad 2: GND -> GND3
- SW4 pad 2: GND -> GND3
- SW5 pad 2: GND -> GND3
- SW6 pad 2: GND -> GND3
- U1 pad 11: GND -> GND3
- U10 pad S: GND -> GND3
- U11 pad S: GND -> GND3
- U12 pad S: GND -> GND3
- U13 pad S: GND -> GND3
- U14 pad S: GND -> GND3
- U15 pad S: GND -> GND3
- U2 pad 11: GND -> GND3
- U21 pad S: GND -> GND3
- U22 pad S: GND -> GND3
- U23 pad S: GND -> GND3
- U24 pad S: GND -> GND3
- U3 pad 11: GND -> GND3
- U4 pad 39: LED8 -> B_LED8
- U4 pad 68: PA9 -> B_PA9
- U4 pad 70: USB_D- -> B_USB_D-
- U4 pad 71: USB_D+ -> B_USB_D+
- U8 pad S: GND -> GND3
- U9 pad S: GND -> GND3
Routing:
- net +3V3: track 341.4 -> 0.00 mm, vias 18 -> 0
- net +12V: track 255.4 -> 0.00 mm, vias 10 -> 0
- net +5V: track 162.2 -> 0.00 mm, vias 2 -> 0
- net 1V25: track 138.8 -> 0.00 mm, vias 2 -> 0
- net AIN6-LED: track 124.6 -> 0.00 mm, vias 6 -> 0
- net -12V: track 111.8 -> 0.00 mm, vias 3 -> 0
- net AIN5-LED: track 108.6 -> 0.00 mm, vias 4 -> 0
- net /DCA/OutA: track 103.8 -> 0.00 mm
- net /DCA/OutB: track 98.2 -> 0.00 mm
- net AIN3: track 93.6 -> 0.00 mm, vias 2 -> 0
- net AIN0-LED: track 91.2 -> 0.00 mm, vias 2 -> 0
- net AIN3-LED: track 88.8 -> 0.00 mm, vias 1 -> 0
- net AIN7: track 88.5 -> 0.00 mm
- net AIN7-LED: track 88.0 -> 0.00 mm, vias 3 -> 0
- net LED0: track 81.7 -> 0.00 mm, vias 1 -> 0
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- added copper zone on B.Cu, net GND3
- added copper zone on F.Cu, net GND3
Other:
- board size 120 x 100 mm -> 120 x 205 mm
- board text added: "WT-V004"
- board text removed: "-12V"
- board text removed: "12V"
- board text removed: "5V"
- board text removed: "GND"
- board text removed: "NC"
- board text removed: "WT-V003"

Commit message: this will be a monster
Parts:
- added C40: C-100nF-0805, Capacitor_SMD:C_0805_2012Metric_Pad1.18x1.45mm_HandSolder, B.Cu at (59.7, -19.9)
- added C41: C-100nF-0805, Capacitor_SMD:C_0805_2012Metric_Pad1.18x1.45mm_HandSolder, B.Cu at (64.0, -19.0)
- added C42: C-Pol-10uF-TAN, Capacitor_Tantalum_SMD:CP_EIA-6032-28_Kemet-C, B.Cu at (52.8, -17.7)
- C29: moved to B.Cu
- C4: moved to F.Cu
- moved C4 184.7 mm to (25.8, -52.5), turned to 180 degrees
- moved C5 149.6 mm to (35.2, -66.6)
- moved C29 123.0 mm to (49.8, -16.3), turned to 90 degrees
- moved J2 114.0 mm to (67.1, -74.1), turned to 180 degrees
- moved C18 113.3 mm to (45.7, -31.8)
- moved C19 113.3 mm to (43.6, -32.2)
- moved C16 113.2 mm to (55.9, -33.5), turned to -90 degrees
- moved U17 112.4 mm to (50.6, -33.9)
- moved U16 108.5 mm to (66.6, -8.58)
- moved C22 106.9 mm to (63.3, -33.2), turned to 180 degrees
- moved C21 106.2 mm to (44.2, -12.9), turned to -90 degrees
- moved U19 105.6 mm to (62.7, -27.4), turned to 180 degrees
- moved C25 105.1 mm to (64.2, -16.0), turned to 0 degrees
- moved JP2 103.6 mm to (47.4, -16.1)
- moved C24 101.2 mm to (56.6, -17.7)
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Connections:
- BackBoard_1 pad 11: unconnected-(BackBoard_1-Pad11) -> B_LED5
- BackBoard_1 pad 13: unconnected-(BackBoard_1-Pad13) -> B_LED4
- BackBoard_1 pad 15: unconnected-(BackBoard_1-Pad15) -> B_LED3
- BackBoard_1 pad 17: unconnected-(BackBoard_1-Pad17) -> B_LED2
- BackBoard_1 pad 19: unconnected-(BackBoard_1-Pad19) -> B_LED1
- BackBoard_1 pad 21: unconnected-(BackBoard_1-Pad21) -> B_LED0
- BackBoard_1 pad 7: unconnected-(BackBoard_1-Pad7) -> B_LED7
- BackBoard_1 pad 9: unconnected-(BackBoard_1-Pad9) -> B_LED6
- FrontBoard_1 pad 11: unconnected-(FrontBoard_1-Pad11) -> LED5
- FrontBoard_1 pad 13: unconnected-(FrontBoard_1-Pad13) -> LED4
- FrontBoard_1 pad 15: unconnected-(FrontBoard_1-Pad15) -> LED3
- FrontBoard_1 pad 17: unconnected-(FrontBoard_1-Pad17) -> LED2
- FrontBoard_1 pad 19: unconnected-(FrontBoard_1-Pad19) -> LED1
- FrontBoard_1 pad 21: unconnected-(FrontBoard_1-Pad21) -> LED0
- FrontBoard_1 pad 7: unconnected-(FrontBoard_1-Pad7) -> LED7
- FrontBoard_1 pad 9: unconnected-(FrontBoard_1-Pad9) -> LED6
- U4 pad 1: LED2 -> B_LED2
- U4 pad 2: LED3 -> B_LED3
- U4 pad 3: LED4 -> B_LED4
- U4 pad 38: LED7 -> B_LED7
- U4 pad 4: LED5 -> B_LED5
- U4 pad 5: LED6 -> B_LED6
- U4 pad 97: LED0 -> B_LED0
- U4 pad 98: LED1 -> B_LED1
Routing:
- net +5V: track 0.00 -> 45.3 mm, vias 0 -> 1
- net +3V3: track 0.00 -> 42.4 mm, vias 0 -> 8
- net GND: track 0.00 -> 38.2 mm, vias 0 -> 5
- net RST: track 0.00 -> 37.5 mm
- net SWDIO: track 0.00 -> 36.9 mm
- net JTDI: track 0.00 -> 28.9 mm
- net TRACESWO: track 0.00 -> 28.4 mm
- net SWDCLK: track 0.00 -> 28.3 mm
- net /DCA/DACA/B: track 0.00 -> 26.7 mm, vias 0 -> 1
- net B_PA9: track 21.9 -> 0.00 mm
- net B_USB_D-: track 21.6 -> 0.04 mm
- net Net-(R1-Pad2): track 0.00 -> 21.4 mm, vias 0 -> 1
- net B_USB_D+: track 18.7 -> 0.04 mm
- net /DCA/CS: track 0.00 -> 16.9 mm, vias 0 -> 1
- net B_LED8: track 0.00 -> 16.7 mm
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- added copper zone on B.Cu, net +3V3
- added copper zone on F.Cu, net +3V3
- added copper zone on In1.Cu, net +3V3
- added copper zone on In2.Cu, net +3V3

Commit message: working on v3 - so far so good
Parts:
- R1, R10, R9: moved to B.Cu
- moved U6 107.0 mm to (58.8, -85.1)
- moved C23 100.4 mm to (36.7, -82.4), turned to 90 degrees
- moved R9 98.0 mm to (42.4, -82.6), turned to 0 degrees
- moved C17 95.5 mm to (53.0, -82.3), turned to 90 degrees
- moved R11 94.9 mm to (48.4, -82.2), turned to -90 degrees
- moved C9 94.9 mm to (40.3, -78.5)
- moved U5 93.8 mm to (42.5, -85.1)
- moved R10 92.8 mm to (58.8, -82.6), turned to 0 degrees
- moved C8 89.9 mm to (56.6, -78.5), turned to 180 degrees
- moved R12 89.8 mm to (64.8, -82.2), turned to -90 degrees
Connections:
- BackBoard_1 pad 1: B_USB_D+ -> unconnected-(BackBoard_1-Pad1)
- BackBoard_1 pad 2: B_USB_D- -> unconnected-(BackBoard_1-Pad2)
- BackBoard_1 pad 23: unconnected-(BackBoard_1-Pad23) -> B_OutB
- BackBoard_1 pad 25: unconnected-(BackBoard_1-Pad25) -> B_OutA
- BackBoard_1 pad 27: unconnected-(BackBoard_1-Pad27) -> B_USB_D+
- BackBoard_1 pad 28: unconnected-(BackBoard_1-Pad28) -> B_USB_D-
- FrontBoard_1 pad 1: USB_D+ -> unconnected-(FrontBoard_1-Pad1)
- FrontBoard_1 pad 2: USB_D- -> unconnected-(FrontBoard_1-Pad2)
- FrontBoard_1 pad 23: unconnected-(FrontBoard_1-Pad23) -> OutB
- FrontBoard_1 pad 25: unconnected-(FrontBoard_1-Pad25) -> OutA
- FrontBoard_1 pad 27: unconnected-(FrontBoard_1-Pad27) -> USB_D+
- FrontBoard_1 pad 28: unconnected-(FrontBoard_1-Pad28) -> USB_D-
- Out_1 pad S: GND -> GND3
- Out_1 pad T: /DCA/OutA -> OutA
- Out_1 pad TN: /DCA/OutA -> OutA
- Out_2 pad S: GND -> GND3
- Out_2 pad T: /DCA/OutB -> OutB
- Out_2 pad TN: /DCA/OutB -> OutB
- R11 pad 2: /DCA/OutA -> B_OutA
- R12 pad 2: /DCA/OutB -> B_OutB
- U5 pad 1: /DCA/OutA -> B_OutA
- U6 pad 1: /DCA/OutB -> B_OutB
Routing:
- net B_LED3: track 0.00 -> 105.9 mm, vias 0 -> 1
- net B_LED4: track 0.00 -> 103.6 mm, vias 0 -> 1
- net B_LED5: track 0.00 -> 100.8 mm, vias 0 -> 1
- net B_LED6: track 0.00 -> 99.9 mm, vias 0 -> 1
- net B_LED0: track 0.00 -> 99.4 mm, vias 0 -> 1
- net B_LED2: track 0.00 -> 99.1 mm, vias 0 -> 1
- net B_LED1: track 0.00 -> 98.1 mm, vias 0 -> 1
- net OutB: track 0.00 -> 87.6 mm
- net OutA: track 0.00 -> 74.8 mm
- net B_LED7: track 6.48 -> 61.7 mm, vias 0 -> 1
- net /DCA/InB: track 0.00 -> 51.8 mm, vias 0 -> 3
- net /DCA/InA: track 0.00 -> 45.1 mm, vias 0 -> 1
- net B_LED8: track 16.7 -> 60.1 mm
- net B_OutB: track 0.00 -> 40.3 mm, vias 0 -> 1
- net Net-(U5-Pad8): track 0.00 -> 35.6 mm
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