File: tlc.kicad_sch (KiCad schematic)
At the start: 15 parts, among them U5 TL074, U6 TL074, U7 TLC7528

Commit message: wip v3
Parts:
- gave numbers to parts that had none: 2
Changed lines of the file:
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@@
   (symbol (lib_id "eurorack:C-100nF-0805") (at 273.685 35.56 0) (unit 1)
     (in_bom yes) (on_board yes)
-    (property "Reference" "C?" (id 0) (at 274.32 33.02 0)
+    (property "Reference" "C28" (id 0) (at 274.32 33.02 0)
       (effects (font (size 1.27 1.27)) (justify left))
     )
@@
   (symbol (lib_id "power:GND") (at 235.585 31.115 0) (unit 1)
     (in_bom yes) (on_board yes) (fields_autoplaced)
-    (property "Reference" "#PWR?" (id 0) (at 235.585 37.465 0)
+    (property "Reference" "#PWR0167" (id 0) (at 235.585 37.465 0)
       (effects (font (size 1.27 1.27)) hide)
     )
@@
   (symbol (lib_id "eurorack:C-100nF-0805") (at 240.665 35.56 0) (unit 1)
     (in_bom yes) (on_board yes)
-    (property "Reference" "C?" (id 0) (at 241.3 33.02 0)
+    (property "Reference" "C20" (id 0) (at 241.3 33.02 0)
       (effects (font (size 1.27 1.27)) (justify left))
     )
@@
   (symbol (lib_id "power:GND") (at 278.765 30.48 0) (unit 1)
     (in_bom yes) (on_board yes) (fields_autoplaced)
-    (property "Reference" "#PWR?" (id 0) (at 278.765 36.83 0)
-      (effects (font (size 1.27 1.27)) hide)
-    )
+    (property "Reference" "#PWR0166" (id 0) (at 278.765 36.83 0)
+      (effects (font (size 1.27 1.27)) hide)
+    )
