File: wt.kicad_sch (KiCad schematic)
At the start: 16 parts, among them U4 STM32F407VGTx, Y1 Crystal_8Mhz

Commit message: New design
Connections:
- net AIN4: now also U4.34 (PC5); no longer U4.31 (PA6)
- net AIN5: now also U4.33 (PC4); no longer U4.32 (PA7)
- net AIN6: now also U4.32 (PA7); no longer U4.33 (PC4)
- net AIN7: now also U4.31 (PA6); no longer U4.34 (PC5)
Changed lines of the file:
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@@
     )
   )
-  (global_label "AIN7" (shape input) (at 210.185 194.31 0) (fields_autoplaced)
-    (effects (font (size 1.27 1.27)) (justify left))
-    (property "Intersheet References" "${INTERSHEET_REFS}" (id 0) (at 216.8314 194.2306 0)
+  (global_label "AIN7" (shape input) (at 210.185 110.49 0) (fields_autoplaced)
+    (effects (font (size 1.27 1.27)) (justify left))
+    (property "Intersheet References" "${INTERSHEET_REFS}" (id 0) (at 216.8314 110.4106 0)
       (effects (font (size 1.27 1.27)) (justify left) hide)
     )
@@
     )
   )
-  (global_label "AIN6" (shape input) (at 210.185 191.77 0) (fields_autoplaced)
-    (effects (font (size 1.27 1.27)) (justify left))
-    (property "Intersheet References" "${INTERSHEET_REFS}" (id 0) (at 216.8314 191.6906 0)
+  (global_label "AIN6" (shape input) (at 210.185 113.03 0) (fields_autoplaced)
+    (effects (font (size 1.27 1.27)) (justify left))
+    (property "Intersheet References" "${INTERSHEET_REFS}" (id 0) (at 216.8314 112.9506 0)
       (effects (font (size 1.27 1.27)) (justify left) hide)
     )
@@
     )
   )
-  (global_label "AIN5" (shape input) (at 210.185 113.03 0) (fields_autoplaced)
-    (effects (font (size 1.27 1.27)) (justify left))
-    (property "Intersheet References" "${INTERSHEET_REFS}" (id 0) (at 216.8314 112.9506 0)
+  (global_label "AIN5" (shape input) (at 210.185 191.77 0) (fields_autoplaced)
+    (effects (font (size 1.27 1.27)) (justify left))
+    (property "Intersheet References" "${INTERSHEET_REFS}" (id 0) (at 216.8314 191.6906 0)
       (effects (font (size 1.27 1.27)) (justify left) hide)
     )
@@
     )
   )
-  (global_label "AIN4" (shape input) (at 210.185 110.49 0) (fields_autoplaced)
-    (effects (font (size 1.27 1.27)) (justify left))
-    (property "Intersheet References" "${INTERSHEET_REFS}" (id 0) (at 216.8314 110.4106 0)
+  (global_label "AIN4" (shape input) (at 210.185 194.31 0) (fields_autoplaced)
+    (effects (font (size 1.27 1.27)) (justify left))
+    (property "Intersheet References" "${INTERSHEET_REFS}" (id 0) (at 216.8314 194.2306 0)
       (effects (font (size 1.27 1.27)) (justify left) hide)
     )
@@
       (reference "#PWR0114") (unit 1) (value "GND") (footprint "")
     )
+    (path "/e824c659-32ba-400c-8fa0-3368d4abf8c1/30f04acf-723c-4d3e-94a4-a5f0e6d178d3"
+      (reference "#PWR0115") (unit 1) (value "+5V") (footprint "")
+    )
+    (path "/e824c659-32ba-400c-8fa0-3368d4abf8c1/8ac53db2-d6e6-4bae-90d5-f1663d2ec3f8"
+      (reference "#PWR0116") (unit 1) (value "+12V") (footprint "")
+    )
+    (path "/e824c659-32ba-400c-8fa0-3368d4abf8c1/a36b1143-6afb-42b8-af03-718868cb1657"
+      (reference "#PWR0117") (unit 1) (value "GND") (footprint "")
+    )
+    (path "/e824c659-32ba-400c-8fa0-3368d4abf8c1/8e1fc2a4-6bc8-4cac-90b8-f11a9ab0fe25"
+      (reference "#PWR0118") (unit 1) (value "-12V") (footprint "")
+    )
     (path "/ce04e4c1-9ead-4ae1-8ff7-69cbf5a77bba"
       (reference "C1") (unit 1) (value "C-22pF-0805") (footprint "Capacitor_SMD:C_0805_2012Metric_Pad1.18x1.45mm_HandSolder")
@@
       (reference "C23") (unit 1) (value "C-100nF-0805") (footprint "Capacitor_SMD:C_0805_2012Metric_Pad1.18x1.45mm_HandSolder")
     )
+    (path "/e824c659-32ba-400c-8fa0-3368d4abf8c1/176f5890-fa87-445d-a5eb-8d285f6782ca"
+      (reference "C24") (unit 1) (value "C-Pol-10uF-TAN") (footprint "Capacitor_Tantalum_SMD:CP_EIA-6032-28_Kemet-C")
+    )
+    (path "/e824c659-32ba-400c-8fa0-3368d4abf8c1/37f200f9-d47d-4193-b313-0b39d00ccfb3"
+      (reference "C25") (unit 1) (value "C-Pol-10uF-TAN") (footprint "Capacitor_Tantalum_SMD:CP_EIA-6032-28_Kemet-C")
+    )
     (path "/a4608a5e-e243-4c2c-8818-85504544b9cc/d0672bd5-77fe-44f2-986e-5c9230ada444/4f91f338-1b66-422c-86de-03e72a556e0f"
       (reference "D1") (unit 1) (value "BAS 85 VIS") (footprint "Diode_SMD:D_MiniMELF")
@@
       (reference "JP1") (unit 1) (value "BOOT0") (footprint "Connector_PinHeader_2.54mm:PinHeader_1x03_P2.54mm_Vertical")
     )
+    (path "/e824c659-32ba-400c-8fa0-3368d4abf8c1/62791df6-a75e-4c5d-b235-9ee523a71715"
+      (reference "JP2") (unit 1) (value "Jumper_2_Open") (footprint "Jumper:SolderJumper-2_P1.3mm_Open_Pad1.0x1.5mm")
+    )
     (path "/c5361e3e-2aef-494b-b75e-964fb5c67e4f"
       (reference "Out_1") (unit 1) (value "LUM-1502-03_3.5mm_mono_vertical_jack") (footprint "eurorack:LUM 1502-03")
@@
       (reference "U15") (unit 1) (value "LUM-1502-03_3.5mm_mono_vertical_jack") (footprint "eurorack:LUM 1502-03")
     )
-    (path "/e824c659-32ba-400c-8fa0-3368d4abf8c1/0110dc09-7260-4b72-824b-88272648f7c3"
-      (reference "U16") (unit 1) (value "power_conn_10") (footprint "eurorack:power_10")
+    (path "/e824c659-32ba-400c-8fa0-3368d4abf8c1/28d25066-cbcd-4827-8d73-23d9cf8fcee8"
+      (reference "U16") (unit 1) (value "power_conn_16") (footprint "eurorack:power_16")
     )
     (path "/e824c659-32ba-400c-8fa0-3368d4abf8c1/a45fefe3-f07e-4ab0-9207-a515cd2966e0"
       (reference "U17") (unit 1) (value "REF191") (footprint "Package_SO:SO-8_3.9x4.9mm_P1.27mm")
     )
-    (path "/e824c659-32ba-400c-8fa0-3368d4abf8c1/4698fe25-be48-4bd9-9c3f-bff9cceafc29"
-      (reference "U18") (unit 1) (value "L78L05ACU") (footprint "Package_TO_SOT_SMD:SOT-89-3_Handsoldering")
+    (path "/e824c659-32ba-400c-8fa0-3368d4abf8c1/42d93df4-449e-4283-8eae-f718a193e111"
+      (reference "U18") (unit 1) (value "LM7805_TO220") (footprint "Package_TO_SOT_THT:TO-220-3_Vertical")
     )
     (path "/e824c659-32ba-400c-8fa0-3368d4abf8c1/885721f2-5906-4c87-b7c5-9a9ae02f9855"

Commit message: yet an other new version with 3 boards
Parts:
- added BackBoard_1: Conn_01x28_Female, Connector_PinSocket_2.54mm:PinSocket_2x14_P2.54mm_Vertical, symbol Connector:Conn_01x28_Female
- added BackBoard_2, BackBoard_3: Conn_01x14_Male, Connector_PinHeader_2.54mm:PinHeader_1x14_P2.54mm_Vertical, symbol Connector:Conn_01x14_Male
- added FrontBoard_1: Conn_01x28_Male, Connector_PinHeader_2.54mm:PinHeader_2x14_P2.54mm_Vertical, symbol Connector:Conn_01x28_Male
- added FrontBoard_2, FrontBoard_3: Conn_01x14_Female, Connector_PinSocket_2.54mm:PinSocket_1x14_P2.54mm_Vertical, symbol Connector:Conn_01x14_Female
Connections:
- net GND: now also BackBoard_1.3 (Pin_3)
- net LED8: now also FrontBoard_1.5 (Pin_5); no longer U4.39 (PE8)
- net PA9: now also FrontBoard_1.4 (Pin_4); no longer U4.68 (PA9)
- net USB_D+: now also FrontBoard_1.1 (Pin_1); no longer U4.71 (PA12)
- net USB_D-: now also FrontBoard_1.2 (Pin_2); no longer U4.70 (PA11)
- new net B_LED8: BackBoard_1.5 (Pin_5), U4.39 (PE8)
- new net B_PA9: BackBoard_1.4 (Pin_4), U4.68 (PA9)
- new net B_USB_D+: BackBoard_1.1 (Pin_1), U4.71 (PA12)
- new net B_USB_D-: BackBoard_1.2 (Pin_2), U4.70 (PA11)
- new net GND3: FrontBoard_1.3 (Pin_3)

Commit message: this will be a monster
Connections:
- net LED0: now also FrontBoard_1.21 (Pin_21); no longer U4.97 (PE0)
- net LED1: now also FrontBoard_1.19 (Pin_19); no longer U4.98 (PE1)
- net LED2: now also FrontBoard_1.17 (Pin_17); no longer U4.1 (PE2)
- net LED3: now also FrontBoard_1.15 (Pin_15); no longer U4.2 (PE3)
- net LED4: now also FrontBoard_1.13 (Pin_13); no longer U4.3 (PE4)
- net LED5: now also FrontBoard_1.11 (Pin_11); no longer U4.4 (PE5)
- net LED6: now also FrontBoard_1.9 (Pin_9); no longer U4.5 (PE6)
- net LED7: now also FrontBoard_1.7 (Pin_7); no longer U4.38 (PE7)
- net B_LED5: now reaches BackBoard_1.11 (Pin_11)
- net B_LED5: now also U4.4 (PE5)
- net B_LED4: now reaches BackBoard_1.13 (Pin_13)
- net B_LED4: now also U4.3 (PE4)
- net B_LED3: now reaches BackBoard_1.15 (Pin_15)
- net B_LED3: now also U4.2 (PE3)
- net B_LED2: now reaches BackBoard_1.17 (Pin_17)
- net B_LED2: now also U4.1 (PE2)
- net B_LED1: now reaches BackBoard_1.19 (Pin_19)
- net B_LED1: now also U4.98 (PE1)
- net B_LED0: now reaches BackBoard_1.21 (Pin_21)
- net B_LED0: now also U4.97 (PE0)
- net B_LED7: now reaches BackBoard_1.7 (Pin_7)
- net B_LED7: now also U4.38 (PE7)
- net B_LED6: now reaches BackBoard_1.9 (Pin_9)
- net B_LED6: now also U4.5 (PE6)

Commit message: working on v3 - so far so good
Connections:
- net DCA/OutA is gone; now on net OutA: Out_1.T, Out_1.TN
- net DCA/OutB is gone; now on net OutB: Out_2.T, Out_2.TN
- net B_USB_D+: now also BackBoard_1.27 (Pin_27); no longer BackBoard_1.1 (Pin_1)
- net B_USB_D-: now also BackBoard_1.28 (Pin_28); no longer BackBoard_1.2 (Pin_2)
- net GND: no longer Out_1.S, Out_2.S
- net GND3: now also Out_1.S, Out_2.S
- net USB_D+: now also FrontBoard_1.27 (Pin_27); no longer FrontBoard_1.1 (Pin_1)
- net USB_D-: now also FrontBoard_1.28 (Pin_28); no longer FrontBoard_1.2 (Pin_2)
- net B_OutB: now reaches BackBoard_1.23 (Pin_23)
- net B_OutA: now reaches BackBoard_1.25 (Pin_25)
- net OutB: now reaches FrontBoard_1.23 (Pin_23)
- net OutA: now reaches FrontBoard_1.25 (Pin_25)
Other:
- moved on the sheet: Out_1
