File: power.kicad_sch (KiCad schematic)
At the start: 22 parts, among them U16 power_conn_16, U17 REF191, U18 LM7805_TO220, U19 ZLDO1117G33TA

Commit message: wip led panel
Parts:
- gave numbers to parts that had none: 9
Changed lines of the file:
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@@
   (symbol (lib_id "eurorack:C-100nF-0805") (at 156.845 68.58 0) (unit 1)
     (in_bom yes) (on_board yes)
-    (property "Reference" "C?" (id 0) (at 157.48 66.04 0)
+    (property "Reference" "C36" (id 0) (at 157.48 66.04 0)
       (effects (font (size 1.27 1.27)) (justify left))
     )
@@
   (symbol (lib_id "eurorack:C-100nF-0805") (at 133.985 36.195 0) (unit 1)
     (in_bom yes) (on_board yes)
-    (property "Reference" "C?" (id 0) (at 134.62 33.655 0)
+    (property "Reference" "C31" (id 0) (at 134.62 33.655 0)
       (effects (font (size 1.27 1.27)) (justify left))
     )
@@
   (symbol (lib_id "eurorack:C-100nF-0805") (at 151.13 68.58 0) (unit 1)
     (in_bom yes) (on_board yes)
-    (property "Reference" "C?" (id 0) (at 151.765 66.04 0)
+    (property "Reference" "C35" (id 0) (at 151.765 66.04 0)
       (effects (font (size 1.27 1.27)) (justify left))
     )
@@
   (symbol (lib_id "eurorack:C-100nF-0805") (at 83.185 69.85 0) (unit 1)
     (in_bom yes) (on_board yes)
-    (property "Reference" "C?" (id 0) (at 83.82 67.31 0)
+    (property "Reference" "C29" (id 0) (at 83.82 67.31 0)
       (effects (font (size 1.27 1.27)) (justify left))
     )
@@
   (symbol (lib_id "eurorack:C-100nF-0805") (at 138.43 97.79 0) (unit 1)
     (in_bom yes) (on_board yes)
-    (property "Reference" "C?" (id 0) (at 139.065 95.25 0)
+    (property "Reference" "C32" (id 0) (at 139.065 95.25 0)
       (effects (font (size 1.27 1.27)) (justify left))
     )
@@
   (symbol (lib_id "eurorack:C-100nF-0805") (at 104.14 68.58 0) (unit 1)
     (in_bom yes) (on_board yes)
-    (property "Reference" "C?" (id 0) (at 104.775 66.04 0)
+    (property "Reference" "C30" (id 0) (at 104.775 66.04 0)
       (effects (font (size 1.27 1.27)) (justify left))
     )
@@
   (symbol (lib_id "power:+5V") (at 138.43 92.71 0) (unit 1)
     (in_bom yes) (on_board yes) (fields_autoplaced)
-    (property "Reference" "#PWR?" (id 0) (at 138.43 96.52 0)
+    (property "Reference" "#PWR0121" (id 0) (at 138.43 96.52 0)
       (effects (font (size 1.27 1.27)) hide)
     )
@@
   (symbol (lib_id "power:GND") (at 151.13 74.93 0) (unit 1)
     (in_bom yes) (on_board yes) (fields_autoplaced)
-    (property "Reference" "#PWR?" (id 0) (at 151.13 81.28 0)
+    (property "Reference" "#PWR0119" (id 0) (at 151.13 81.28 0)
       (effects (font (size 1.27 1.27)) hide)
     )
@@
   (symbol (lib_id "eurorack:C-100nF-0805") (at 139.065 68.58 0) (unit 1)
     (in_bom yes) (on_board yes)
-    (property "Reference" "C?" (id 0) (at 139.7 66.04 0)
+    (property "Reference" "C33" (id 0) (at 139.7 66.04 0)
       (effects (font (size 1.27 1.27)) (justify left))
     )
@@
   (symbol (lib_id "power:GND") (at 138.43 102.87 0) (unit 1)
     (in_bom yes) (on_board yes) (fields_autoplaced)
-    (property "Reference" "#PWR?" (id 0) (at 138.43 109.22 0)
+    (property "Reference" "#PWR0122" (id 0) (at 138.43 109.22 0)
       (effects (font (size 1.27 1.27)) hide)
     )
@@
   (symbol (lib_id "power:+3V3") (at 151.13 62.865 0) (unit 1)
     (in_bom yes) (on_board yes) (fields_autoplaced)
-    (property "Reference" "#PWR?" (id 0) (at 151.13 66.675 0)
+    (property "Reference" "#PWR0120" (id 0) (at 151.13 66.675 0)
       (effects (font (size 1.27 1.27)) hide)
     )
@@
   (symbol (lib_id "eurorack:C-100nF-0805") (at 145.415 68.58 0) (unit 1)
     (in_bom yes) (on_board yes)
-    (property "Reference" "C?" (id 0) (at 146.05 66.04 0)
+    (property "Reference" "C34" (id 0) (at 146.05 66.04 0)
       (effects (font (size 1.27 1.27)) (justify left))
     )
@@
   (symbol (lib_id "eurorack:C-100nF-0805") (at 73.66 36.195 0) (unit 1)
     (in_bom yes) (on_board yes)
-    (property "Reference" "C?" (id 0) (at 74.295 33.655 0)
-      (effects (font (size 1.27 1.27)) (justify left))
-    )
+    (property "Reference" "C28" (id 0) (at 74.295 33.655 0)
+      (effects (font (size 1.27 1.27)) (justify left))
+    )

Commit message: this will be a monster
Parts:
- added C40, C41: C-100nF-0805, Capacitor_SMD:C_0805_2012Metric_Pad1.18x1.45mm_HandSolder, symbol eurorack:C-100nF-0805
- added C42: C-Pol-10uF-TAN, Capacitor_Tantalum_SMD:CP_EIA-6032-28_Kemet-C, symbol eurorack:C-Pol-10uF-TAN
Connections:
- net +12V: now also C40.1
- net +5V: now also C42.1
- net -12V: now also C41.2
- net GND: now also C40.2, C41.1, C42.2
Changed lines of the file:
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@@
   (junction (at 109.855 43.18) (diameter 0) (color 0 0 0 0)
   )
+  (junction (at 79.375 60.96) (diameter 0) (color 0 0 0 0)
+  )
+  (junction (at 82.55 88.9) (diameter 0) (color 0 0 0 0)
+  )
   (junction (at 151.13 64.77) (diameter 0) (color 0 0 0 0)
   )
@@
   (junction (at 104.14 60.96) (diameter 0) (color 0 0 0 0)
   )
+  (junction (at 82.55 107.95) (diameter 0) (color 0 0 0 0)
+  )
   (junction (at 79.375 28.575) (diameter 0) (color 0 0 0 0)
   )
@@
   (junction (at 151.13 72.39) (diameter 0) (color 0 0 0 0)
   )
+  (junction (at 77.47 99.06) (diameter 0) (color 0 0 0 0)
+  )
   (junction (at 46.99 76.2) (diameter 0) (color 0 0 0 0)
   )
@@
   (junction (at 82.55 99.06) (diameter 0) (color 0 0 0 0)
   )
+  (junction (at 83.185 75.565) (diameter 0) (color 0 0 0 0)
+  )
   (junction (at 109.855 28.575) (diameter 0) (color 0 0 0 0)
   )
@@
   )
   (junction (at 46.99 91.44) (diameter 0) (color 0 0 0 0)
+  )
+  (junction (at 71.755 99.06) (diameter 0) (color 0 0 0 0)
   )
   (junction (at 64.135 83.82) (diameter 0) (color 0 0 0 0)
@@
     (stroke (width 0) (type default) (color 0 0 0 0))
   )
+  (wire (pts (xy 82.55 88.9) (xy 82.55 90.17))
+    (stroke (width 0) (type default) (color 0 0 0 0))
+  )
+  (wire (pts (xy 71.755 107.95) (xy 82.55 107.95))
+    (stroke (width 0) (type default) (color 0 0 0 0))
+  )
   (wire (pts (xy 83.185 60.96) (xy 83.185 66.04))
     (stroke (width 0) (type default) (color 0 0 0 0))
@@
     (stroke (width 0) (type default) (color 0 0 0 0))
   )
+  (wire (pts (xy 76.2 73.66) (xy 76.2 75.565))
+    (stroke (width 0) (type default) (color 0 0 0 0))
+  )
   (wire (pts (xy 90.043 36.195) (xy 90.043 43.18))
     (stroke (width 0) (type default) (color 0 0 0 0))
@@
     (stroke (width 0) (type default) (color 0 0 0 0))
   )
+  (wire (pts (xy 71.755 88.9) (xy 82.55 88.9))
+    (stroke (width 0) (type default) (color 0 0 0 0))
+  )
+  (wire (pts (xy 71.755 97.79) (xy 71.755 99.06))
+    (stroke (width 0) (type default) (color 0 0 0 0))
+  )
   (wire (pts (xy 139.065 72.39) (xy 145.415 72.39))
     (stroke (width 0) (type default) (color 0 0 0 0))
@@
     (stroke (width 0) (type default) (color 0 0 0 0))
   )
+  (wire (pts (xy 71.755 99.06) (xy 71.755 100.33))
+    (stroke (width 0) (type default) (color 0 0 0 0))
+  )
   (wire (pts (xy 77.47 100.33) (xy 77.47 99.06))
     (stroke (width 0) (type default) (color 0 0 0 0))
@@
     (stroke (width 0) (type default) (color 0 0 0 0))
   )
-  (wire (pts (xy 82.55 87.63) (xy 82.55 90.17))
+  (wire (pts (xy 82.55 87.63) (xy 82.55 88.9))
     (stroke (width 0) (type default) (color 0 0 0 0))
   )
@@
     (stroke (width 0) (type default) (color 0 0 0 0))
   )
+  (wire (pts (xy 76.2 60.96) (xy 79.375 60.96))
+    (stroke (width 0) (type default) (color 0 0 0 0))
+  )
   (wire (pts (xy 151.13 72.39) (xy 151.13 74.93))
     (stroke (width 0) (type default) (color 0 0 0 0))
@@
     (stroke (width 0) (type default) (color 0 0 0 0))
   )
+  (wire (pts (xy 76.2 66.04) (xy 76.2 60.96))
+    (stroke (width 0) (type default) (color 0 0 0 0))
+  )
   (wire (pts (xy 83.185 73.66) (xy 83.185 75.565))
     (stroke (width 0) (type default) (color 0 0 0 0))
@@
     (stroke (width 0) (type default) (color 0 0 0 0))
   )
+  (wire (pts (xy 71.755 90.17) (xy 71.755 88.9))
+    (stroke (width 0) (type default) (color 0 0 0 0))
+  )
   (wire (pts (xy 33.02 76.2) (xy 46.99 76.2))
     (stroke (width 0) (type default) (color 0 0 0 0))
@@
   )
   (wire (pts (xy 104.14 60.96) (xy 109.855 60.96))
+    (stroke (width 0) (type default) (color 0 0 0 0))
+  )
+  (wire (pts (xy 76.2 75.565) (xy 83.185 75.565))
+    (stroke (width 0) (type default) (color 0 0 0 0))
+  )
+  (wire (pts (xy 71.755 99.06) (xy 77.47 99.06))
     (stroke (width 0) (type default) (color 0 0 0 0))
   )
@@
     (pin "1")
   )
+  (symbol (lib_id "eurorack:C-Pol-10uF-TAN") (at 76.2 69.85 0) (unit 1)
+    (in_bom yes) (on_board yes) (fields_autoplaced)
+    (property "Reference" "C42" (id 0) (at 80.01 67.6909 0)
+      (effects (font (size 1.27 1.27)) (justify left))
+    )
+    (property "Value" "C-Pol-10uF-TAN" (id 1) (at 80.01 70.2309 0)
+      (effects (font (size 1.27 1.27)) (justify left))
+    )
+    (property "Footprint" "Capacitor_Tantalum_SMD:CP_EIA-6032-28_Kemet-C" (id 2) (at 77.1652 73.66 0)
+      (effects (font (size 1.27 1.27)) hide)
+    )
+    (property "Datasheet" "https://www.reichelt.at/at/de/smd-tantal-kondensator-10-f-25v-tps-6032-10-25-p167056.html?r=1" (id 3) (at 76.2 69.85 0)
+      (effects (font (size 1.27 1.27)) hide)
+    )
+    (pin "1")
+    (pin "2")
+  )
   (symbol (lib_id "power:+5V") (at 57.277 31.115 0) (unit 1)
     (in_bom yes) (on_board yes) (fields_autoplaced)
@@
     (pin "1")
   )
+  (symbol (lib_id "eurorack:C-100nF-0805") (at 71.755 93.98 0) (unit 1)
+    (in_bom yes) (on_board yes)
+    (property "Reference" "C40" (id 0) (at 72.39 91.44 0)
+      (effects (font (size 1.27 1.27)) (justify left))
+    )
+    (property "Value" "C-100nF-0805" (id 1) (at 68.58 101.6 90)
+      (effects (font (size 1.27 1.27)) (justify left))
+    )
+    (property "Footprint" "Capacitor_SMD:C_0805_2012Metric_Pad1.18x1.45mm_HandSolder" (id 2) (at 72.7202 97.79 0)
+      (effects (font (size 1.27 1.27)) hide)
+    )
+    (property "Datasheet" "https://secure.reichelt.com/at/en/smd-multilayer-ceramic-capacitor-100-n-10--x7r-g0805-100n-p31879.html?&nbc=1" (id 3) (at 71.755 93.98 0)
+      (effects (font (size 1.27 1.27)) hide)
+    )
+    (pin "1")
+    (pin "2")
+  )
   (symbol (lib_id "eurorack:+2V048") (at 64.135 83.82 0) (unit 1)
     (in_bom yes) (on_board yes) (fields_autoplaced)
@@
     (pin "1")
   )
+  (symbol (lib_id "eurorack:C-100nF-0805") (at 71.755 104.14 0) (unit 1)
+    (in_bom yes) (on_board yes)
+    (property "Reference" "C41" (id 0) (at 72.39 101.6 0)
+      (effects (font (size 1.27 1.27)) (justify left))
+    )
+    (property "Value" "C-100nF-0805" (id 1) (at 68.58 118.745 90)
+      (effects (font (size 1.27 1.27)) (justify left))
+    )
+    (property "Footprint" "Capacitor_SMD:C_0805_2012Metric_Pad1.18x1.45mm_HandSolder" (id 2) (at 72.7202 107.95 0)
+      (effects (font (size 1.27 1.27)) hide)
+    )
+    (property "Datasheet" "https://secure.reichelt.com/at/en/smd-multilayer-ceramic-capacitor-100-n-10--x7r-g0805-100n-p31879.html?&nbc=1" (id 3) (at 71.755 104.14 0)
+      (effects (font (size 1.27 1.27)) hide)
+    )
+    (pin "1")
+    (pin "2")
+  )
   (symbol (lib_id "eurorack:C-100nF-0805") (at 73.66 36.195 0) (unit 1)

Commit message: wip
Parts:
- removed C20: C-Pol-10uF-TAN, Capacitor_Tantalum_SMD:CP_EIA-6032-28_Kemet-C, symbol eurorack:C-Pol-10uF-TAN
- removed C28: C-100nF-0805, Capacitor_SMD:C_0805_2012Metric_Pad1.18x1.45mm_HandSolder, symbol eurorack:C-100nF-0805
Changed lines of the file:
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@@
   (junction (at 82.55 107.95) (diameter 0) (color 0 0 0 0)
   )
-  (junction (at 79.375 28.575) (diameter 0) (color 0 0 0 0)
-  )
-  (junction (at 90.043 43.18) (diameter 0) (color 0 0 0 0)
-  )
   (junction (at 104.14 75.565) (diameter 0) (color 0 0 0 0)
   )
@@
   )
   (junction (at 33.02 83.82) (diameter 0) (color 0 0 0 0)
-  )
-  (junction (at 79.375 43.18) (diameter 0) (color 0 0 0 0)
   )
   (junction (at 46.99 91.44) (diameter 0) (color 0 0 0 0)
@@
     (stroke (width 0) (type default) (color 0 0 0 0))
   )
-  (wire (pts (xy 79.375 28.575) (xy 79.375 32.385))
-    (stroke (width 0) (type default) (color 0 0 0 0))
-  )
   (wire (pts (xy 151.13 72.39) (xy 156.845 72.39))
     (stroke (width 0) (type default) (color 0 0 0 0))
@@
     (stroke (width 0) (type default) (color 0 0 0 0))
   )
-  (wire (pts (xy 73.66 28.575) (xy 79.375 28.575))
-    (stroke (width 0) (type default) (color 0 0 0 0))
-  )
   (wire (pts (xy 100.33 60.96) (xy 104.14 60.96))
     (stroke (width 0) (type default) (color 0 0 0 0))
@@
     (stroke (width 0) (type default) (color 0 0 0 0))
   )
-  (wire (pts (xy 79.375 43.18) (xy 90.043 43.18))
-    (stroke (width 0) (type default) (color 0 0 0 0))
-  )
   (wire (pts (xy 107.823 28.575) (xy 109.855 28.575))
     (stroke (width 0) (type default) (color 0 0 0 0))
@@
     (stroke (width 0) (type default) (color 0 0 0 0))
   )
-  (wire (pts (xy 73.66 43.18) (xy 79.375 43.18))
-    (stroke (width 0) (type default) (color 0 0 0 0))
-  )
   (wire (pts (xy 109.855 43.18) (xy 133.985 43.18))
     (stroke (width 0) (type default) (color 0 0 0 0))
@@
     (stroke (width 0) (type default) (color 0 0 0 0))
   )
-  (wire (pts (xy 73.66 32.385) (xy 73.66 28.575))
-    (stroke (width 0) (type default) (color 0 0 0 0))
-  )
   (wire (pts (xy 79.375 28.575) (xy 82.423 28.575))
     (stroke (width 0) (type default) (color 0 0 0 0))
@@
     (stroke (width 0) (type default) (color 0 0 0 0))
   )
-  (wire (pts (xy 79.375 40.005) (xy 79.375 43.18))
-    (stroke (width 0) (type default) (color 0 0 0 0))
-  )
   (wire (pts (xy 52.705 42.545) (xy 58.42 42.545))
     (stroke (width 0) (type default) (color 0 0 0 0))
   )
   (wire (pts (xy 27.305 83.82) (xy 33.02 83.82))
-    (stroke (width 0) (type default) (color 0 0 0 0))
-  )
-  (wire (pts (xy 73.66 40.005) (xy 73.66 43.18))
     (stroke (width 0) (type default) (color 0 0 0 0))
   )
@@
     (pin "1")
   )
-  (symbol (lib_id "eurorack:C-Pol-10uF-TAN") (at 79.375 36.195 0) (unit 1)
-    (in_bom yes) (on_board yes) (fields_autoplaced)
-    (property "Reference" "C20" (id 0) (at 82.55 34.0359 0)
-      (effects (font (size 1.27 1.27)) (justify left))
-    )
-    (property "Value" "C-Pol-10uF-TAN" (id 1) (at 82.55 36.5759 0)
-      (effects (font (size 1.27 1.27)) (justify left))
-    )
-    (property "Footprint" "Capacitor_Tantalum_SMD:CP_EIA-6032-28_Kemet-C" (id 2) (at 80.3402 40.005 0)
-      (effects (font (size 1.27 1.27)) hide)
-    )
-    (property "Datasheet" "https://www.reichelt.at/at/de/smd-tantal-kondensator-10-f-25v-tps-6032-10-25-p167056.html?r=1" (id 3) (at 79.375 36.195 0)
-      (effects (font (size 1.27 1.27)) hide)
-    )
-    (pin "1")
-    (pin "2")
-  )
   (symbol (lib_id "eurorack:C-Pol-1uF-TAN") (at 57.785 87.63 0) (unit 1)
     (in_bom yes) (on_board yes)
@@
       (effects (font (size 1.27 1.27)) hide)
     )
-    (pin "1")
-    (pin "2")
-  )
-  (symbol (lib_id "eurorack:C-100nF-0805") (at 73.66 36.195 0) (unit 1)
-    (in_bom yes) (on_board yes)
-    (property "Reference" "C28" (id 0) (at 74.295 33.655 0)
-      (effects (font (size 1.27 1.27)) (justify left))
-    )
-    (property "Value" "C-100nF-0805" (id 1) (at 70.485 50.8 90)
-      (effects (font (size 1.27 1.27)) (justify left))
-    )
-    (property "Footprint" "Capacitor_SMD:C_0805_2012Metric_Pad1.18x1.45mm_HandSolder" (id 2) (at 74.6252 40.005 0)
-      (effects (font (size 1.27 1.27)) hide)
-    )
-    (property "Datasheet" "https://secure.reichelt.com/at/en/smd-multilayer-ceramic-capacitor-100-n-10--x7r-g0805-100n-p31879.html?&nbc=1" (id 3) (at 73.66 36.195 0)
-      (effects (font (size 1.27 1.27)) hide)
-    )

Commit message: wip v3
Parts:
- added C43: C-100nF-0805, Capacitor_SMD:C_0805_2012Metric_Pad1.18x1.45mm_HandSolder, symbol eurorack:C-100nF-0805
Connections:
- net +3V3: now also C43.1
- net GND: now also C43.2
Changed lines of the file:
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@@
 (kicad_sch (version 20211123) (generator eeschema)
   (paper "A4")
+  (junction (at 156.845 72.39) (diameter 0) (color 0 0 0 0)
+  )
   (junction (at 109.855 43.18) (diameter 0) (color 0 0 0 0)
+  )
+  (junction (at 156.845 64.77) (diameter 0) (color 0 0 0 0)
   )
   (junction (at 79.375 60.96) (diameter 0) (color 0 0 0 0)
@@
     (stroke (width 0) (type default) (color 0 0 0 0))
   )
+  (wire (pts (xy 156.845 64.77) (xy 163.195 64.77))
+    (stroke (width 0) (type default) (color 0 0 0 0))
+  )
   (wire (pts (xy 139.065 72.39) (xy 145.415 72.39))
     (stroke (width 0) (type default) (color 0 0 0 0))
@@
   )
   (wire (pts (xy 109.855 28.575) (xy 133.985 28.575))
+    (stroke (width 0) (type default) (color 0 0 0 0))
+  )
+  (wire (pts (xy 156.845 72.39) (xy 163.195 72.39))
     (stroke (width 0) (type default) (color 0 0 0 0))
   )
@@
       (effects (font (size 1.27 1.27)) hide)
     )
+    (pin "1")
+    (pin "2")
+  )
+  (symbol (lib_id "eurorack:C-100nF-0805") (at 163.195 68.58 0) (unit 1)
+    (in_bom yes) (on_board yes)
+    (property "Reference" "C43" (id 0) (at 163.83 66.04 0)
+      (effects (font (size 1.27 1.27)) (justify left))
+    )
+    (property "Value" "C-100nF-0805" (id 1) (at 160.02 83.185 90)
+      (effects (font (size 1.27 1.27)) (justify left))
+    )
+    (property "Footprint" "Capacitor_SMD:C_0805_2012Metric_Pad1.18x1.45mm_HandSolder" (id 2) (at 164.1602 72.39 0)
+      (effects (font (size 1.27 1.27)) hide)
+    )
+    (property "Datasheet" "https://secure.reichelt.com/at/en/smd-multilayer-ceramic-capacitor-100-n-10--x7r-g0805-100n-p31879.html?&nbc=1" (id 3) (at 163.195 68.58 0)
+      (effects (font (size 1.27 1.27)) hide)
+    )
