File: controls.kicad_sch (KiCad schematic)
At the start: 6 parts, among them U1 LM324, U2 LM324, U3 LM324

Commit message: wip v3
Connections:
- net +3V3 renamed +3.3VA
Changed lines of the file:
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@@
     (pin "2")
+  )
+  (symbol (lib_id "power:+3.3VA") (at 163.195 29.21 0) (unit 1)
+    (in_bom yes) (on_board yes) (fields_autoplaced)
+    (property "Reference" "#PWR?" (id 0) (at 163.195 33.02 0)
+      (effects (font (size 1.27 1.27)) hide)
+    )
+    (property "Value" "+3.3VA" (id 1) (at 163.195 24.13 0))
+    (property "Footprint" "" (id 2) (at 163.195 29.21 0)
+      (effects (font (size 1.27 1.27)) hide)
+    )
+    (property "Datasheet" "" (id 3) (at 163.195 29.21 0)
+      (effects (font (size 1.27 1.27)) hide)
+    )
+    (pin "1")
   )
   (symbol (lib_id "eurorack:LM324") (at 155.575 38.735 0) (unit 5)
@@
       (effects (font (size 1.27 1.27)) hide)
     )
-    (pin "1")
-  )
-  (symbol (lib_id "power:+3V3") (at 163.195 29.21 0) (unit 1)
-    (in_bom yes) (on_board yes) (fields_autoplaced)
-    (property "Reference" "#PWR094" (id 0) (at 163.195 33.02 0)
-      (effects (font (size 1.27 1.27)) hide)
-    )
-    (property "Value" "+3V3" (id 1) (at 163.195 24.13 0))
-    (property "Footprint" "" (id 2) (at 163.195 29.21 0)
-      (effects (font (size 1.27 1.27)) hide)
-    )
-    (property "Datasheet" "" (id 3) (at 163.195 29.21 0)
-      (effects (font (size 1.27 1.27)) hide)
-    )
