File: pot.kicad_sch (KiCad schematic)
At the start: 7 parts, among them U12 LUM-1502-03_3.5mm_mono_vertic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, U2 LM324

Commit message: working on the PCB
Parts:
- renumbered D5 to D1, R27 to R15, R28 to R16, R29 to R17, RV5 to RV1, U2 to U1, U12 to U8
Changed lines of the file:
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@@
     (effects (font (size 1.27 1.27)) (justify left))
   )
-  (symbol (lib_id "eurorack:LUM-1502-03_3.5mm_mono_vertical_jack") (at 33.655 67.31 0) (mirror x)
+  (symbol (lib_id "eurorack:LUM-1502-03_3.5mm_mono_vertical_jack") (at 33.655 67.31 0) (mirror x) (unit 1)
     (in_bom yes) (on_board yes) (fields_autoplaced)
-    (property "Reference" "U12" (id 0) (at 28.575 65.4049 0)
+    (property "Reference" "U8" (id 0) (at 28.575 65.4049 0)
       (effects (font (size 1.27 1.27)) (justify right))
     )
@@
     (pin "TN")
   )
-  (symbol (lib_id "eurorack:LM324") (at 88.265 63.5 0) (mirror x)
+  (symbol (lib_id "eurorack:LM324") (at 88.265 63.5 0) (mirror x) (unit 1)
     (in_bom yes) (on_board yes) (fields_autoplaced)
-    (property "Reference" "U2" (id 0) (at 88.265 53.34 0))
+    (property "Reference" "U1" (id 0) (at 88.265 53.34 0))
     (property "Value" "LM324" (id 1) (at 88.265 55.88 0))
     (property "Footprint" "Package_SO:SO-14_3.9x8.65mm_P1.27mm" (id 2) (at 86.995 66.04 0)
@@
     (pin "2")
     (pin "3")
+    (pin "5")
+    (pin "6")
+    (pin "7")
+    (pin "10")
+    (pin "8")
+    (pin "9")
+    (pin "12")
+    (pin "13")
+    (pin "14")
+    (pin "11")
+    (pin "4")
   )
-  (symbol (lib_id "power:GND") (at 39.37 71.12 0) (mirror y)
+  (symbol (lib_id "power:GND") (at 39.37 71.12 0) (mirror y) (unit 1)
     (in_bom yes) (on_board yes) (fields_autoplaced)
-    (property "Reference" "#PWR0112" (id 0) (at 39.37 77.47 0)
+    (property "Reference" "#PWR033" (id 0) (at 39.37 77.47 0)
       (effects (font (size 1.27 1.27)) hide)
     )
@@
     (pin "1")
   )
-  (symbol (lib_id "eurorack:BAS 85 VIS") (at 47.625 66.04 180)
+  (symbol (lib_id "eurorack:BAS 85 VIS") (at 47.625 66.04 180) (unit 1)
     (in_bom yes) (on_board yes) (fields_autoplaced)
-    (property "Reference" "D5" (id 0) (at 47.625 59.055 0))
+    (property "Reference" "D1" (id 0) (at 47.625 59.055 0))
     (property "Value" "BAS 85 VIS" (id 1) (at 47.625 61.595 0))
     (property "Footprint" "Diode_SMD:D_MiniMELF" (id 2) (at 47.625 61.595 0)
@@
     (pin "2")
   )
-  (symbol (lib_id "power:GND") (at 102.87 76.2 0)
+  (symbol (lib_id "power:GND") (at 102.87 76.2 0) (unit 1)
     (in_bom yes) (on_board yes) (fields_autoplaced)
-    (property "Reference" "#PWR0114" (id 0) (at 102.87 82.55 0)
+    (property "Reference" "#PWR035" (id 0) (at 102.87 82.55 0)
       (effects (font (size 1.27 1.27)) hide)
     )
@@
     (pin "1")
   )
-  (symbol (lib_id "eurorack:Pot_500") (at 102.87 71.12 0)
+  (symbol (lib_id "eurorack:Pot_500") (at 102.87 71.12 0) (unit 1)
     (in_bom yes) (on_board yes) (fields_autoplaced)
-    (property "Reference" "RV5" (id 0) (at 100.33 69.8499 0)
+    (property "Reference" "RV1" (id 0) (at 100.33 69.8499 0)
       (effects (font (size 1.27 1.27)) (justify right))
     )
@@
     (pin "3")
   )
-  (symbol (lib_id "eurorack:R-2k-0805") (at 68.58 69.85 0)
+  (symbol (lib_id "eurorack:R-2k-0805") (at 68.58 69.85 0) (unit 1)
     (in_bom yes) (on_board yes) (fields_autoplaced)
-    (property "Reference" "R29" (id 0) (at 71.12 68.5799 0)
+    (property "Reference" "R17" (id 0) (at 71.12 68.5799 0)
       (effects (font (size 1.27 1.27)) (justify left))
     )
@@
     (pin "2")
   )
-  (symbol (lib_id "eurorack:R-2k-0805") (at 39.37 54.61 0)
+  (symbol (lib_id "eurorack:R-2k-0805") (at 39.37 54.61 0) (unit 1)
     (in_bom yes) (on_board yes) (fields_autoplaced)
-    (property "Reference" "R27" (id 0) (at 41.91 53.3399 0)
+    (property "Reference" "R15" (id 0) (at 41.91 53.3399 0)
       (effects (font (size 1.27 1.27)) (justify left))
     )
@@
     (pin "2")
   )
-  (symbol (lib_id "power:+12V") (at 39.37 49.53 0)
+  (symbol (lib_id "power:+12V") (at 39.37 49.53 0) (unit 1)
     (in_bom yes) (on_board yes) (fields_autoplaced)
-    (property "Reference" "#PWR0111" (id 0) (at 39.37 53.34 0)
+    (property "Reference" "#PWR032" (id 0) (at 39.37 53.34 0)
       (effects (font (size 1.27 1.27)) hide)
     )
@@
     (pin "1")
   )
-  (symbol (lib_id "power:GND") (at 68.58 75.565 0)
+  (symbol (lib_id "power:GND") (at 68.58 75.565 0) (unit 1)
     (in_bom yes) (on_board yes) (fields_autoplaced)
-    (property "Reference" "#PWR0113" (id 0) (at 68.58 81.915 0)
+    (property "Reference" "#PWR034" (id 0) (at 68.58 81.915 0)
       (effects (font (size 1.27 1.27)) hide)
     )
@@
     (pin "1")
   )
-  (symbol (lib_id "eurorack:R-7k5-0805") (at 60.325 66.04 90)
+  (symbol (lib_id "eurorack:R-7k5-0805") (at 60.325 66.04 90) (unit 1)
     (in_bom yes) (on_board yes) (fields_autoplaced)
-    (property "Reference" "R28" (id 0) (at 60.325 59.69 90))
+    (property "Reference" "R16" (id 0) (at 60.325 59.69 90))
     (property "Value" "R-7k5-0805" (id 1) (at 60.325 62.23 90))
     (property "Footprint" "Resistor_SMD:R_0805_2012Metric" (id 2) (at 60.325 67.818 90)

Commit message: Working on the PCB / JTAG
Parts:
- renumbered D1 to D30, R15 to R78, R16 to R79, R17 to R80, RV1 to RV13, U8 to U24, U1 to U3
Changed lines of the file:
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@@
     (effects (font (size 1.27 1.27)) (justify left))
   )
-  (symbol (lib_id "eurorack:LUM-1502-03_3.5mm_mono_vertical_jack") (at 33.655 67.31 0) (mirror x) (unit 1)
+  (symbol (lib_id "eurorack:LUM-1502-03_3.5mm_mono_vertical_jack") (at 33.655 67.31 0) (mirror x)
     (in_bom yes) (on_board yes) (fields_autoplaced)
-    (property "Reference" "U8" (id 0) (at 28.575 65.4049 0)
+    (property "Reference" "U24" (id 0) (at 28.575 65.4049 0)
       (effects (font (size 1.27 1.27)) (justify right))
     )
@@
     (pin "TN")
   )
-  (symbol (lib_id "eurorack:LM324") (at 88.265 63.5 0) (mirror x) (unit 1)
+  (symbol (lib_id "eurorack:LM324") (at 88.265 63.5 0) (mirror x)
     (in_bom yes) (on_board yes) (fields_autoplaced)
-    (property "Reference" "U1" (id 0) (at 88.265 53.34 0))
+    (property "Reference" "U3" (id 0) (at 88.265 53.34 0))
     (property "Value" "LM324" (id 1) (at 88.265 55.88 0))
     (property "Footprint" "Package_SO:SO-14_3.9x8.65mm_P1.27mm" (id 2) (at 86.995 66.04 0)
@@
     (pin "2")
     (pin "3")
-    (pin "5")
-    (pin "6")
-    (pin "7")
-    (pin "10")
-    (pin "8")
-    (pin "9")
-    (pin "12")
-    (pin "13")
-    (pin "14")
-    (pin "11")
-    (pin "4")
   )
-  (symbol (lib_id "power:GND") (at 39.37 71.12 0) (mirror y) (unit 1)
+  (symbol (lib_id "power:GND") (at 39.37 71.12 0) (mirror y)
     (in_bom yes) (on_board yes) (fields_autoplaced)
-    (property "Reference" "#PWR033" (id 0) (at 39.37 77.47 0)
+    (property "Reference" "#PWR0112" (id 0) (at 39.37 77.47 0)
       (effects (font (size 1.27 1.27)) hide)
     )
@@
     (pin "1")
   )
-  (symbol (lib_id "eurorack:BAS 85 VIS") (at 47.625 66.04 180) (unit 1)
+  (symbol (lib_id "eurorack:BAS 85 VIS") (at 47.625 66.04 180)
     (in_bom yes) (on_board yes) (fields_autoplaced)
-    (property "Reference" "D1" (id 0) (at 47.625 59.055 0))
+    (property "Reference" "D30" (id 0) (at 47.625 59.055 0))
     (property "Value" "BAS 85 VIS" (id 1) (at 47.625 61.595 0))
     (property "Footprint" "Diode_SMD:D_MiniMELF" (id 2) (at 47.625 61.595 0)
@@
     (pin "2")
   )
-  (symbol (lib_id "power:GND") (at 102.87 76.2 0) (unit 1)
+  (symbol (lib_id "power:GND") (at 102.87 76.2 0)
     (in_bom yes) (on_board yes) (fields_autoplaced)
-    (property "Reference" "#PWR035" (id 0) (at 102.87 82.55 0)
+    (property "Reference" "#PWR0114" (id 0) (at 102.87 82.55 0)
       (effects (font (size 1.27 1.27)) hide)
     )
@@
     (pin "1")
   )
-  (symbol (lib_id "eurorack:Pot_500") (at 102.87 71.12 0) (unit 1)
+  (symbol (lib_id "eurorack:Pot_500") (at 102.87 71.12 0)
     (in_bom yes) (on_board yes) (fields_autoplaced)
-    (property "Reference" "RV1" (id 0) (at 100.33 69.8499 0)
+    (property "Reference" "RV13" (id 0) (at 100.33 69.8499 0)
       (effects (font (size 1.27 1.27)) (justify right))
     )
@@
     (pin "3")
   )
-  (symbol (lib_id "eurorack:R-2k-0805") (at 68.58 69.85 0) (unit 1)
+  (symbol (lib_id "eurorack:R-2k-0805") (at 68.58 69.85 0)
     (in_bom yes) (on_board yes) (fields_autoplaced)
-    (property "Reference" "R17" (id 0) (at 71.12 68.5799 0)
+    (property "Reference" "R80" (id 0) (at 71.12 68.5799 0)
       (effects (font (size 1.27 1.27)) (justify left))
     )
@@
     (pin "2")
   )
-  (symbol (lib_id "eurorack:R-2k-0805") (at 39.37 54.61 0) (unit 1)
+  (symbol (lib_id "eurorack:R-2k-0805") (at 39.37 54.61 0)
     (in_bom yes) (on_board yes) (fields_autoplaced)
-    (property "Reference" "R15" (id 0) (at 41.91 53.3399 0)
+    (property "Reference" "R78" (id 0) (at 41.91 53.3399 0)
       (effects (font (size 1.27 1.27)) (justify left))
     )
@@
     (pin "2")
   )
-  (symbol (lib_id "power:+12V") (at 39.37 49.53 0) (unit 1)
+  (symbol (lib_id "power:+12V") (at 39.37 49.53 0)
     (in_bom yes) (on_board yes) (fields_autoplaced)
-    (property "Reference" "#PWR032" (id 0) (at 39.37 53.34 0)
+    (property "Reference" "#PWR0111" (id 0) (at 39.37 53.34 0)
       (effects (font (size 1.27 1.27)) hide)
     )
@@
     (pin "1")
   )
-  (symbol (lib_id "power:GND") (at 68.58 75.565 0) (unit 1)
+  (symbol (lib_id "power:GND") (at 68.58 75.565 0)
     (in_bom yes) (on_board yes) (fields_autoplaced)
-    (property "Reference" "#PWR034" (id 0) (at 68.58 81.915 0)
+    (property "Reference" "#PWR0113" (id 0) (at 68.58 81.915 0)
       (effects (font (size 1.27 1.27)) hide)
     )
@@
     (pin "1")
   )
-  (symbol (lib_id "eurorack:R-7k5-0805") (at 60.325 66.04 90) (unit 1)
+  (symbol (lib_id "eurorack:R-7k5-0805") (at 60.325 66.04 90)
     (in_bom yes) (on_board yes) (fields_autoplaced)
-    (property "Reference" "R16" (id 0) (at 60.325 59.69 90))
+    (property "Reference" "R79" (id 0) (at 60.325 59.69 90))
     (property "Value" "R-7k5-0805" (id 1) (at 60.325 62.23 90))
     (property "Footprint" "Resistor_SMD:R_0805_2012Metric" (id 2) (at 60.325 67.818 90)

Commit message: final touches
Parts:
- renumbered D30 to D1, R78 to R15, R79 to R16, R80 to R17, RV13 to RV1, U3 to U1, U24 to U8
Changed lines of the file:
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@@
     (effects (font (size 1.27 1.27)) (justify left))
   )
-  (symbol (lib_id "eurorack:LUM-1502-03_3.5mm_mono_vertical_jack") (at 33.655 67.31 0) (mirror x)
+  (symbol (lib_id "eurorack:LUM-1502-03_3.5mm_mono_vertical_jack") (at 33.655 67.31 0) (mirror x) (unit 1)
     (in_bom yes) (on_board yes) (fields_autoplaced)
-    (property "Reference" "U24" (id 0) (at 28.575 65.4049 0)
+    (property "Reference" "U8" (id 0) (at 28.575 65.4049 0)
       (effects (font (size 1.27 1.27)) (justify right))
     )
@@
     (pin "TN")
   )
-  (symbol (lib_id "eurorack:LM324") (at 88.265 63.5 0) (mirror x)
+  (symbol (lib_id "eurorack:LM324") (at 88.265 63.5 0) (mirror x) (unit 1)
     (in_bom yes) (on_board yes) (fields_autoplaced)
-    (property "Reference" "U3" (id 0) (at 88.265 53.34 0))
+    (property "Reference" "U1" (id 0) (at 88.265 53.34 0))
     (property "Value" "LM324" (id 1) (at 88.265 55.88 0))
     (property "Footprint" "Package_SO:SO-14_3.9x8.65mm_P1.27mm" (id 2) (at 86.995 66.04 0)
@@
     (pin "2")
     (pin "3")
+    (pin "5")
+    (pin "6")
+    (pin "7")
+    (pin "10")
+    (pin "8")
+    (pin "9")
+    (pin "12")
+    (pin "13")
+    (pin "14")
+    (pin "11")
+    (pin "4")
   )
-  (symbol (lib_id "power:GND") (at 39.37 71.12 0) (mirror y)
+  (symbol (lib_id "power:GND") (at 39.37 71.12 0) (mirror y) (unit 1)
     (in_bom yes) (on_board yes) (fields_autoplaced)
-    (property "Reference" "#PWR0112" (id 0) (at 39.37 77.47 0)
+    (property "Reference" "#PWR033" (id 0) (at 39.37 77.47 0)
       (effects (font (size 1.27 1.27)) hide)
     )
@@
     (pin "1")
   )
-  (symbol (lib_id "eurorack:BAS 85 VIS") (at 47.625 66.04 180)
+  (symbol (lib_id "eurorack:BAS 85 VIS") (at 47.625 66.04 180) (unit 1)
     (in_bom yes) (on_board yes) (fields_autoplaced)
-    (property "Reference" "D30" (id 0) (at 47.625 59.055 0))
+    (property "Reference" "D1" (id 0) (at 47.625 59.055 0))
     (property "Value" "BAS 85 VIS" (id 1) (at 47.625 61.595 0))
     (property "Footprint" "Diode_SMD:D_MiniMELF" (id 2) (at 47.625 61.595 0)
@@
     (pin "2")
   )
-  (symbol (lib_id "power:GND") (at 102.87 76.2 0)
+  (symbol (lib_id "power:GND") (at 102.87 76.2 0) (unit 1)
     (in_bom yes) (on_board yes) (fields_autoplaced)
-    (property "Reference" "#PWR0114" (id 0) (at 102.87 82.55 0)
+    (property "Reference" "#PWR035" (id 0) (at 102.87 82.55 0)
       (effects (font (size 1.27 1.27)) hide)
     )
@@
     (pin "1")
   )
-  (symbol (lib_id "eurorack:Pot_500") (at 102.87 71.12 0)
+  (symbol (lib_id "eurorack:Pot_500") (at 102.87 71.12 0) (unit 1)
     (in_bom yes) (on_board yes) (fields_autoplaced)
-    (property "Reference" "RV13" (id 0) (at 100.33 69.8499 0)
+    (property "Reference" "RV1" (id 0) (at 100.33 69.8499 0)
       (effects (font (size 1.27 1.27)) (justify right))
     )
@@
     (pin "3")
   )
-  (symbol (lib_id "eurorack:R-2k-0805") (at 68.58 69.85 0)
+  (symbol (lib_id "eurorack:R-2k-0805") (at 68.58 69.85 0) (unit 1)
     (in_bom yes) (on_board yes) (fields_autoplaced)
-    (property "Reference" "R80" (id 0) (at 71.12 68.5799 0)
+    (property "Reference" "R17" (id 0) (at 71.12 68.5799 0)
       (effects (font (size 1.27 1.27)) (justify left))
     )
@@
     (pin "2")
   )
-  (symbol (lib_id "eurorack:R-2k-0805") (at 39.37 54.61 0)
+  (symbol (lib_id "eurorack:R-2k-0805") (at 39.37 54.61 0) (unit 1)
     (in_bom yes) (on_board yes) (fields_autoplaced)
-    (property "Reference" "R78" (id 0) (at 41.91 53.3399 0)
+    (property "Reference" "R15" (id 0) (at 41.91 53.3399 0)
       (effects (font (size 1.27 1.27)) (justify left))
     )
@@
     (pin "2")
   )
-  (symbol (lib_id "power:+12V") (at 39.37 49.53 0)
+  (symbol (lib_id "power:+12V") (at 39.37 49.53 0) (unit 1)
     (in_bom yes) (on_board yes) (fields_autoplaced)
-    (property "Reference" "#PWR0111" (id 0) (at 39.37 53.34 0)
+    (property "Reference" "#PWR032" (id 0) (at 39.37 53.34 0)
       (effects (font (size 1.27 1.27)) hide)
     )
@@
     (pin "1")
   )
-  (symbol (lib_id "power:GND") (at 68.58 75.565 0)
+  (symbol (lib_id "power:GND") (at 68.58 75.565 0) (unit 1)
     (in_bom yes) (on_board yes) (fields_autoplaced)
-    (property "Reference" "#PWR0113" (id 0) (at 68.58 81.915 0)
+    (property "Reference" "#PWR034" (id 0) (at 68.58 81.915 0)
       (effects (font (size 1.27 1.27)) hide)
     )
@@
     (pin "1")
   )
-  (symbol (lib_id "eurorack:R-7k5-0805") (at 60.325 66.04 90)
+  (symbol (lib_id "eurorack:R-7k5-0805") (at 60.325 66.04 90) (unit 1)
     (in_bom yes) (on_board yes) (fields_autoplaced)
-    (property "Reference" "R79" (id 0) (at 60.325 59.69 90))
+    (property "Reference" "R16" (id 0) (at 60.325 59.69 90))
     (property "Value" "R-7k5-0805" (id 1) (at 60.325 62.23 90))
     (property "Footprint" "Resistor_SMD:R_0805_2012Metric" (id 2) (at 60.325 67.818 90)

Commit message: reworking with Pot Lights
Parts:
- RV1: footprint Potentiometer_THT:Potentiometer_Piher_PT-10-V10_Vertical -> eurorack:Potentiometer_Piher_PT-10-V10_Vertical
Connections:
- net GND: now also RV1.11 (LED-), RV1.7 (LED-)
- new net: RV1.10 (LED+), RV1.9 (R)
- new net: RV1.5 (R), RV1.6 (LED+)
- new net LED: RV1.4 (R), RV1.8 (R)
Changed lines of the file:
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@@
   (junction (at 98.425 63.5) (diameter 0) (color 0 0 0 0)
   )
+  (junction (at 96.647 87.63) (diameter 0) (color 0 0 0 0)
+  )
+  (junction (at 98.044 69.85) (diameter 0) (color 0 0 0 0)
+  )
+  (junction (at 102.87 91.694) (diameter 0) (color 0 0 0 0)
+  )
   (junction (at 68.58 66.04) (diameter 0) (color 0 0 0 0)
   )
+  (wire (pts (xy 102.87 89.789) (xy 102.87 91.694))
+    (stroke (width 0) (type default) (color 0 0 0 0))
+  )
+  (wire (pts (xy 99.187 72.644) (xy 99.187 75.057))
+    (stroke (width 0) (type default) (color 0 0 0 0))
+  )
+  (wire (pts (xy 99.187 79.883) (xy 98.044 79.883))
+    (stroke (width 0) (type default) (color 0 0 0 0))
+  )
+  (wire (pts (xy 96.647 91.694) (xy 102.87 91.694))
+    (stroke (width 0) (type default) (color 0 0 0 0))
+  )
   (wire (pts (xy 51.435 66.04) (xy 56.515 66.04))
     (stroke (width 0) (type default) (color 0 0 0 0))
@@
     (stroke (width 0) (type default) (color 0 0 0 0))
   )
-  (wire (pts (xy 102.87 63.5) (xy 102.87 67.31))
-    (stroke (width 0) (type default) (color 0 0 0 0))
-  )
   (wire (pts (xy 98.425 57.15) (xy 98.425 63.5))
     (stroke (width 0) (type default) (color 0 0 0 0))
@@
     (stroke (width 0) (type default) (color 0 0 0 0))
   )
+  (wire (pts (xy 99.187 77.597) (xy 96.647 77.597))
+    (stroke (width 0) (type default) (color 0 0 0 0))
+  )
+  (wire (pts (xy 102.87 91.694) (xy 102.87 92.329))
+    (stroke (width 0) (type default) (color 0 0 0 0))
+  )
   (wire (pts (xy 39.37 63.5) (xy 38.735 63.5))
     (stroke (width 0) (type default) (color 0 0 0 0))
@@
     (stroke (width 0) (type default) (color 0 0 0 0))
   )
+  (wire (pts (xy 102.87 63.5) (xy 102.87 67.183))
+    (stroke (width 0) (type default) (color 0 0 0 0))
+  )
+  (wire (pts (xy 96.647 87.63) (xy 96.647 91.694))
+    (stroke (width 0) (type default) (color 0 0 0 0))
+  )
   (wire (pts (xy 98.425 63.5) (xy 102.87 63.5))
     (stroke (width 0) (type default) (color 0 0 0 0))
@@
     (stroke (width 0) (type default) (color 0 0 0 0))
   )
-  (wire (pts (xy 102.87 74.93) (xy 102.87 76.2))
-    (stroke (width 0) (type default) (color 0 0 0 0))
-  )
   (wire (pts (xy 68.58 66.04) (xy 80.645 66.04))
     (stroke (width 0) (type default) (color 0 0 0 0))
   )
+  (wire (pts (xy 99.187 82.677) (xy 99.187 85.09))
+    (stroke (width 0) (type default) (color 0 0 0 0))
+  )
   (wire (pts (xy 38.735 66.04) (xy 43.815 66.04))
     (stroke (width 0) (type default) (color 0 0 0 0))
@@
     (stroke (width 0) (type default) (color 0 0 0 0))
   )
+  (wire (pts (xy 96.647 77.597) (xy 96.647 87.63))
+    (stroke (width 0) (type default) (color 0 0 0 0))
+  )
+  (wire (pts (xy 98.044 69.85) (xy 99.187 69.85))
+    (stroke (width 0) (type default) (color 0 0 0 0))
+  )
+  (wire (pts (xy 98.044 79.883) (xy 98.044 69.85))
+    (stroke (width 0) (type default) (color 0 0 0 0))
+  )
   (wire (pts (xy 39.37 58.42) (xy 39.37 63.5))
     (stroke (width 0) (type default) (color 0 0 0 0))
   )
-  (wire (pts (xy 106.68 71.12) (xy 108.585 71.12))
+  (wire (pts (xy 96.647 87.63) (xy 99.187 87.63))
+    (stroke (width 0) (type default) (color 0 0 0 0))
+  )
+  (wire (pts (xy 106.807 76.2) (xy 109.728 76.2))
+    (stroke (width 0) (type default) (color 0 0 0 0))
+  )
+  (wire (pts (xy 95.377 69.85) (xy 98.044 69.85))
     (stroke (width 0) (type default) (color 0 0 0 0))
   )
@@
     (stroke (width 0) (type default) (color 0 0 0 0))
   )
-  (hierarchical_label "Out" (shape output) (at 108.585 71.12 0)
+  (hierarchical_label "Out" (shape output) (at 109.728 76.2 0)
     (effects (font (size 1.27 1.27)) (justify left))
+  )
+  (hierarchical_label "LED" (shape input) (at 95.377 69.85 180)
+    (effects (font (size 1.27 1.27)) (justify right))
   )
   (symbol (lib_id "eurorack:LUM-1502-03_3.5mm_mono_vertical_jack") (at 33.655 67.31 0) (mirror x) (unit 1)
@@
     (pin "2")
   )
-  (symbol (lib_id "power:GND") (at 102.87 76.2 0) (unit 1)
-    (in_bom yes) (on_board yes) (fields_autoplaced)
-    (property "Reference" "#PWR035" (id 0) (at 102.87 82.55 0)
-      (effects (font (size 1.27 1.27)) hide)
-    )
-    (property "Value" "GND" (id 1) (at 102.87 80.645 0))
-    (property "Footprint" "" (id 2) (at 102.87 76.2 0)
-      (effects (font (size 1.27 1.27)) hide)
-    )
-    (property "Datasheet" "" (id 3) (at 102.87 76.2 0)
-      (effects (font (size 1.27 1.27)) hide)
-    )
-    (pin "1")
-  )
-  (symbol (lib_id "eurorack:Pot_500") (at 102.87 71.12 0) (unit 1)
-    (in_bom yes) (on_board yes) (fields_autoplaced)
-    (property "Reference" "RV1" (id 0) (at 100.33 69.8499 0)
+  (symbol (lib_id "power:GND") (at 102.87 92.329 0) (unit 1)
+    (in_bom yes) (on_board yes) (fields_autoplaced)
+    (property "Reference" "#PWR035" (id 0) (at 102.87 98.679 0)
+      (effects (font (size 1.27 1.27)) hide)
+    )
+    (property "Value" "GND" (id 1) (at 102.87 96.774 0))
+    (property "Footprint" "" (id 2) (at 102.87 92.329 0)
+      (effects (font (size 1.27 1.27)) hide)
+    )
+    (property "Datasheet" "" (id 3) (at 102.87 92.329 0)
+      (effects (font (size 1.27 1.27)) hide)
+    )
+    (pin "1")
+  )
+  (symbol (lib_id "eurorack:Pot_500") (at 102.997 78.994 0) (unit 1)
+    (in_bom yes) (on_board yes)
+    (property "Reference" "RV1" (id 0) (at 108.966 69.977 0)
       (effects (font (size 1.27 1.27)) (justify right))
     )
-    (property "Value" "Pot_500" (id 1) (at 100.33 72.3899 0)
+    (property "Value" "Pot_500" (id 1) (at 113.411 71.882 0)
       (effects (font (size 1.27 1.27)) (justify right))
     )
-    (property "Footprint" "Potentiometer_THT:Potentiometer_Piher_PT-10-V10_Vertical" (id 2) (at 102.87 71.12 0)
-      (effects (font (size 1.27 1.27)) hide)
-    )
-    (property "Datasheet" "https://secure.reichelt.com/at/en/rotary-potentiometer-500-ohm-linear-4-mm-pih-smc10v10501-p232483.html?&trstct=pos_4&nbc=1" (id 3) (at 102.87 71.12 0)
-      (effects (font (size 1.27 1.27)) hide)
-    )
-    (pin "1")
+    (property "Footprint" "eurorack:Potentiometer_Piher_PT-10-V10_Vertical" (id 2) (at 102.997 78.994 0)
+      (effects (font (size 1.27 1.27)) hide)
+    )
+    (property "Datasheet" "https://secure.reichelt.at/at/en/rotary-potentiometer-500-ohm-linear-4-mm-pih-smc10v10501-p232483.html" (id 3) (at 102.997 78.994 0)
+      (effects (font (size 1.27 1.27)) hide)
+    )
+    (pin "1")
+    (pin "10")
+    (pin "11")
     (pin "2")
     (pin "3")
+    (pin "4")
+    (pin "5")
+    (pin "6")
+    (pin "7")
+    (pin "8")
+    (pin "9")
   )
   (symbol (lib_id "eurorack:R-2k-0805") (at 68.58 69.85 0) (unit 1)
