File: pot.kicad_sch (KiCad schematic)
At the start: 7 parts, among them U1 LM324, U8 LUM-1502-03_3.5mm_mono_vertic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

Commit message: yet an other new version with 3 boards
Connections:
- net GND renamed GND3
Changed lines of the file:
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@@
     (pin "4")
-  )
-  (symbol (lib_id "power:GND") (at 39.37 71.12 0) (mirror y) (unit 1)
-    (in_bom yes) (on_board yes) (fields_autoplaced)
-    (property "Reference" "#PWR033" (id 0) (at 39.37 77.47 0)
-      (effects (font (size 1.27 1.27)) hide)
-    )
-    (property "Value" "GND" (id 1) (at 39.37 76.2 0))
-    (property "Footprint" "" (id 2) (at 39.37 71.12 0)
-      (effects (font (size 1.27 1.27)) hide)
-    )
-    (property "Datasheet" "" (id 3) (at 39.37 71.12 0)
-      (effects (font (size 1.27 1.27)) hide)
-    )
-    (pin "1")
   )
   (symbol (lib_id "eurorack:BAS 85 VIS") (at 47.625 66.04 180) (unit 1)
@@
     (pin "2")
   )
-  (symbol (lib_id "power:GND") (at 102.87 92.329 0) (unit 1)
+  (symbol (lib_id "power:GND3") (at 102.87 92.329 0) (unit 1)
     (in_bom yes) (on_board yes) (fields_autoplaced)
-    (property "Reference" "#PWR035" (id 0) (at 102.87 98.679 0)
+    (property "Reference" "#PWR0106" (id 0) (at 102.87 98.679 0)
       (effects (font (size 1.27 1.27)) hide)
     )
-    (property "Value" "GND" (id 1) (at 102.87 96.774 0))
+    (property "Value" "GND3" (id 1) (at 102.87 97.79 0))
     (property "Footprint" "" (id 2) (at 102.87 92.329 0)
       (effects (font (size 1.27 1.27)) hide)
     )
     (property "Datasheet" "" (id 3) (at 102.87 92.329 0)
+      (effects (font (size 1.27 1.27)) hide)
+    )
+    (pin "1")
+  )
+  (symbol (lib_id "power:GND3") (at 68.58 75.565 0) (unit 1)
+    (in_bom yes) (on_board yes) (fields_autoplaced)
+    (property "Reference" "#PWR0105" (id 0) (at 68.58 81.915 0)
+      (effects (font (size 1.27 1.27)) hide)
+    )
+    (property "Value" "GND3" (id 1) (at 68.58 80.01 0))
+    (property "Footprint" "" (id 2) (at 68.58 75.565 0)
+      (effects (font (size 1.27 1.27)) hide)
+    )
+    (property "Datasheet" "" (id 3) (at 68.58 75.565 0)
       (effects (font (size 1.27 1.27)) hide)
     )
@@
     (pin "8")
     (pin "9")
+  )
+  (symbol (lib_id "power:GND3") (at 39.37 71.12 0) (unit 1)
+    (in_bom yes) (on_board yes) (fields_autoplaced)
+    (property "Reference" "#PWR0108" (id 0) (at 39.37 77.47 0)
+      (effects (font (size 1.27 1.27)) hide)
+    )
+    (property "Value" "GND3" (id 1) (at 39.37 76.2 0))
+    (property "Footprint" "" (id 2) (at 39.37 71.12 0)
+      (effects (font (size 1.27 1.27)) hide)
+    )
+    (property "Datasheet" "" (id 3) (at 39.37 71.12 0)
+      (effects (font (size 1.27 1.27)) hide)
+    )
+    (pin "1")
   )
   (symbol (lib_id "eurorack:R-2k-0805") (at 68.58 69.85 0) (unit 1)
@@
       (effects (font (size 1.27 1.27)) hide)
     )
-    (pin "1")
-  )
-  (symbol (lib_id "power:GND") (at 68.58 75.565 0) (unit 1)
-    (in_bom yes) (on_board yes) (fields_autoplaced)
-    (property "Reference" "#PWR034" (id 0) (at 68.58 81.915 0)
-      (effects (font (size 1.27 1.27)) hide)
-    )
-    (property "Value" "GND" (id 1) (at 68.58 80.01 0))
-    (property "Footprint" "" (id 2) (at 68.58 75.565 0)
-      (effects (font (size 1.27 1.27)) hide)
-    )
-    (property "Datasheet" "" (id 3) (at 68.58 75.565 0)
-      (effects (font (size 1.27 1.27)) hide)
-    )

Commit message: wip v3
Connections:
- net +12V renamed +12VA
Changed lines of the file:
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@@
     (pin "TN")
+  )
+  (symbol (lib_id "power:+12VA") (at 39.37 49.53 0) (unit 1)
+    (in_bom yes) (on_board yes) (fields_autoplaced)
+    (property "Reference" "#PWR?" (id 0) (at 39.37 53.34 0)
+      (effects (font (size 1.27 1.27)) hide)
+    )
+    (property "Value" "+12VA" (id 1) (at 39.37 44.45 0))
+    (property "Footprint" "" (id 2) (at 39.37 49.53 0)
+      (effects (font (size 1.27 1.27)) hide)
+    )
+    (property "Datasheet" "" (id 3) (at 39.37 49.53 0)
+      (effects (font (size 1.27 1.27)) hide)
+    )
+    (pin "1")
   )
   (symbol (lib_id "eurorack:LM324") (at 88.265 63.5 0) (mirror x) (unit 1)
@@
     (pin "2")
   )
-  (symbol (lib_id "power:+12V") (at 39.37 49.53 0) (unit 1)
-    (in_bom yes) (on_board yes) (fields_autoplaced)
-    (property "Reference" "#PWR032" (id 0) (at 39.37 53.34 0)
-      (effects (font (size 1.27 1.27)) hide)
-    )
-    (property "Value" "+12V" (id 1) (at 39.37 43.815 0))
-    (property "Footprint" "" (id 2) (at 39.37 49.53 0)
-      (effects (font (size 1.27 1.27)) hide)
-    )
-    (property "Datasheet" "" (id 3) (at 39.37 49.53 0)
-      (effects (font (size 1.27 1.27)) hide)
-    )
-    (pin "1")
-  )
   (symbol (lib_id "eurorack:R-7k5-0805") (at 60.325 66.04 90) (unit 1)
